Commit message: 去掉hardware中的测试程序

File: src/zhishu_robot_moveit_config/config/zhishu_robot.ros2_control.xacro (robot description, xacro)
@@ -10,4 +10,48 @@
                 <plugin>es_motor_hardware/EsMotorHardwareInterface</plugin>
             </hardware>
+            <!-- right_arm -->
+            <joint name="right_shoulder_pitch_joint">
+                <command_interface name="position"/>
+                <state_interface name="position">
+                  <param name="initial_value">${initial_positions['right_shoulder_pitch_joint']}</param>
+                </state_interface>
+            </joint>
+            <joint name="right_shoulder_roll_joint">
+                <command_interface name="position"/>
+                <state_interface name="position">
+                  <param name="initial_value">${initial_positions['right_shoulder_roll_joint']}</param>
+                </state_interface>
+            </joint>
+            <joint name="right_shoulder_yaw_joint">
+                <command_interface name="position"/>
+                <state_interface name="position">
+                  <param name="initial_value">${initial_positions['right_shoulder_yaw_joint']}</param>
+                </state_interface>
+            </joint>
+            <joint name="right_elbow_pitch_joint">
+                <command_interface name="position"/>
+                <state_interface name="position">
+                  <param name="initial_value">${initial_positions['right_elbow_pitch_joint']}</param>
+                </state_interface>
+            </joint>
+            <joint name="right_wrist_yaw_joint">
+                <command_interface name="position"/>
+                <state_interface name="position">
+                  <param name="initial_value">${initial_positions['right_wrist_yaw_joint']}</param>
+                </state_interface>
+            </joint>
+            <joint name="right_wrist_pitch_joint">
+                <command_interface name="position"/>
+                <state_interface name="position">
+                  <param name="initial_value">${initial_positions['right_wrist_pitch_joint']}</param>
+                </state_interface>
+            </joint>
+            <joint name="right_wrist_roll_joint">
+                <command_interface name="position"/>
+                <state_interface name="position">
+                  <param name="initial_value">${initial_positions['right_wrist_roll_joint']}</param>
+                </state_interface>
+            </joint>
+            <!-- left_arm -->
             <joint name="left_shoulder_pitch_joint">
                 <command_interface name="position"/>
@@ -52,46 +96,4 @@
                 </state_interface>
             </joint>
-            <joint name="right_shoulder_pitch_joint">
-                <command_interface name="position"/>
-                <state_interface name="position">
-                  <param name="initial_value">${initial_positions['right_shoulder_pitch_joint']}</param>
-                </state_interface>
-            </joint>
-            <joint name="right_shoulder_roll_joint">
-                <command_interface name="position"/>
-                <state_interface name="position">
-                  <param name="initial_value">${initial_positions['right_shoulder_roll_joint']}</param>
-                </state_interface>
-            </joint>
-            <joint name="right_shoulder_yaw_joint">
-                <command_interface name="position"/>
-                <state_interface name="position">
-                  <param name="initial_value">${initial_positions['right_shoulder_yaw_joint']}</param>
-                </state_interface>
-            </joint>
-            <joint name="right_elbow_pitch_joint">
-                <command_interface name="position"/>
-                <state_interface name="position">
-                  <param name="initial_value">${initial_positions['right_elbow_pitch_joint']}</param>
-                </state_interface>
-            </joint>
-            <joint name="right_wrist_yaw_joint">
-                <command_interface name="position"/>
-                <state_interface name="position">
-                  <param name="initial_value">${initial_positions['right_wrist_yaw_joint']}</param>
-                </state_interface>
-            </joint>
-            <joint name="right_wrist_pitch_joint">
-                <command_interface name="position"/>
-                <state_interface name="position">
-                  <param name="initial_value">${initial_positions['right_wrist_pitch_joint']}</param>
-                </state_interface>
-            </joint>
-            <joint name="right_wrist_roll_joint">
-                <command_interface name="position"/>
-                <state_interface name="position">
-                  <param name="initial_value">${initial_positions['right_wrist_roll_joint']}</param>
-                </state_interface>
-            </joint>
             <joint name="gripper_left_finger_joint">
                 <command_interface name="position"/>
