Commit message: adapt rk3588

File: src/zhishu_robot_moveit_config/config/zhishu_robot.left_arm.ros2_control.xacro (robot description, xacro)
@@ -1,5 +1,5 @@
 <?xml version="1.0"?>
 <robot xmlns:xacro="http://www.ros.org/wiki/xacro">
-    <xacro:macro name="zhishu_robot_left_arm_ros2_control" params="name initial_positions_file use_gazebo:=false use_fake_hardware:=true">
+    <xacro:macro name="zhishu_robot_left_arm_ros2_control" params="name initial_positions_file use_gazebo:=false use_fake_hardware:=true enable_motors_on_activate:=true">
         <xacro:property name="initial_positions" value="${xacro.load_yaml(initial_positions_file)['initial_positions']}"/>
         <ros2_control name="${name}" type="system">
@@ -18,8 +18,9 @@
                 </xacro:unless>
                 <!-- IgH EtherCAT / GH1 SERVOPACK defaults. Per-joint params below can override these. -->
-                <param name="cycle_ns">2000000</param>
+                <param name="cycle_ns">1000000</param>
                 <param name="enable_dc">true</param>
                 <param name="assign_activate">0x0300</param>
-                <param name="sync0_shift_ns">1000000</param>
+                <!-- Trigger SYNC0 halfway through the 1 ms application cycle. -->
+                <param name="sync0_shift_ns">500000</param>
                 <param name="select_dc_reference_clock">true</param>
                 <param name="dc_reference_alias">0</param>
@@ -27,4 +28,6 @@
                 <param name="enable_realtime">true</param>
                 <param name="realtime_priority">85</param>
+                <param name="realtime_cpu">4</param>
+                <param name="enable_motors_on_activate">${enable_motors_on_activate}</param>
                 <param name="master_index">0</param>
                 <param name="alias">0</param>

File: src/zhishu_robot_moveit_config/config/zhishu_robot.right_arm.ros2_control.xacro (robot description, xacro)
@@ -1,5 +1,5 @@
 <?xml version="1.0"?>
 <robot xmlns:xacro="http://www.ros.org/wiki/xacro">
-    <xacro:macro name="zhishu_robot_right_arm_ros2_control" params="name initial_positions_file use_gazebo:=false use_fake_hardware:=true">
+    <xacro:macro name="zhishu_robot_right_arm_ros2_control" params="name initial_positions_file use_gazebo:=false use_fake_hardware:=true enable_motors_on_activate:=true">
         <xacro:property name="initial_positions" value="${xacro.load_yaml(initial_positions_file)['initial_positions']}"/>
         <ros2_control name="${name}" type="system">
@@ -18,8 +18,9 @@
                 </xacro:unless>
                 <!-- IgH EtherCAT / GH1 SERVOPACK defaults. Per-joint params below can override these. -->
-                <param name="cycle_ns">2000000</param>
+                <param name="cycle_ns">1000000</param>
                 <param name="enable_dc">true</param>
                 <param name="assign_activate">0x0300</param>
-                <param name="sync0_shift_ns">1000000</param>
+                <!-- Trigger SYNC0 halfway through the 1 ms application cycle. -->
+                <param name="sync0_shift_ns">500000</param>
                 <param name="select_dc_reference_clock">true</param>
                 <param name="dc_reference_alias">0</param>
@@ -27,4 +28,6 @@
                 <param name="enable_realtime">true</param>
                 <param name="realtime_priority">85</param>
+                <param name="realtime_cpu">5</param>
+                <param name="enable_motors_on_activate">${enable_motors_on_activate}</param>
                 <param name="master_index">1</param>
                 <param name="alias">0</param>

File: src/zhishu_robot_moveit_config/config/zhishu_robot.urdf.xacro (robot description, xacro)
@@ -4,4 +4,5 @@
     <xacro:arg name="use_gazebo" default="false" />
     <xacro:arg name="use_fake_hardware" default="true" />
+    <xacro:arg name="enable_motors_on_activate" default="true" />
     <!-- Import zhishu_robot urdf file -->
     <xacro:include filename="$(find zhishu_robot_description)/urdf/zhishu_robot.urdf.xacro" />
@@ -14,9 +15,11 @@
             name="LeftArmSystem"
             initial_positions_file="$(arg initial_positions_file)"
-            use_fake_hardware="$(arg use_fake_hardware)"/>
+            use_fake_hardware="$(arg use_fake_hardware)"
+            enable_motors_on_activate="$(arg enable_motors_on_activate)"/>
         <xacro:zhishu_robot_right_arm_ros2_control
             name="RightArmSystem"
             initial_positions_file="$(arg initial_positions_file)"
-            use_fake_hardware="$(arg use_fake_hardware)"/>
+            use_fake_hardware="$(arg use_fake_hardware)"
+            enable_motors_on_activate="$(arg enable_motors_on_activate)"/>
     </xacro:unless>
     <xacro:if value="$(arg use_gazebo)">

Commit message: feat(moveit): 关闭启动阶段 PDO 自动采集

File: src/zhishu_robot_moveit_config/config/zhishu_robot.left_arm.ros2_control.xacro (robot description, xacro)
@@ -1,5 +1,5 @@
 <?xml version="1.0"?>
 <robot xmlns:xacro="http://www.ros.org/wiki/xacro">
-    <xacro:macro name="zhishu_robot_left_arm_ros2_control" params="name initial_positions_file use_gazebo:=false use_fake_hardware:=true enable_motors_on_activate:=true">
+    <xacro:macro name="zhishu_robot_left_arm_ros2_control" params="name initial_positions_file use_gazebo:=false use_fake_hardware:=true enable_motors_on_activate:=true pdo_diagnostics_auto_start:=true">
         <xacro:property name="initial_positions" value="${xacro.load_yaml(initial_positions_file)['initial_positions']}"/>
         <ros2_control name="${name}" type="system">
@@ -35,7 +35,7 @@
                      non-realtime CSV writer. 16384 cycles tolerate a 16 s disk stall. -->
                 <param name="pdo_diagnostics_buffer_cycles">16384</param>
-                <!-- Capture a bounded 20 s startup window even if the ROS service
-                     executor is unavailable. This avoids unbounded disk growth. -->
-                <param name="pdo_diagnostics_auto_start">true</param>
+                <!-- Optionally capture a bounded 20 s startup window even if the ROS
+                     service executor is unavailable. -->
+                <param name="pdo_diagnostics_auto_start">${pdo_diagnostics_auto_start}</param>
                 <param name="pdo_diagnostics_max_cycles">20000</param>
                 <param name="enable_motors_on_activate">${enable_motors_on_activate}</param>

File: src/zhishu_robot_moveit_config/config/zhishu_robot.right_arm.ros2_control.xacro (robot description, xacro)
@@ -1,5 +1,5 @@
 <?xml version="1.0"?>
 <robot xmlns:xacro="http://www.ros.org/wiki/xacro">
-    <xacro:macro name="zhishu_robot_right_arm_ros2_control" params="name initial_positions_file use_gazebo:=false use_fake_hardware:=true enable_motors_on_activate:=true">
+    <xacro:macro name="zhishu_robot_right_arm_ros2_control" params="name initial_positions_file use_gazebo:=false use_fake_hardware:=true enable_motors_on_activate:=true pdo_diagnostics_auto_start:=true">
         <xacro:property name="initial_positions" value="${xacro.load_yaml(initial_positions_file)['initial_positions']}"/>
         <ros2_control name="${name}" type="system">
@@ -35,7 +35,7 @@
                      non-realtime CSV writer. 16384 cycles tolerate a 16 s disk stall. -->
                 <param name="pdo_diagnostics_buffer_cycles">16384</param>
-                <!-- Capture a bounded 20 s startup window even if the ROS service
-                     executor is unavailable. This avoids unbounded disk growth. -->
-                <param name="pdo_diagnostics_auto_start">true</param>
+                <!-- Optionally capture a bounded 20 s startup window even if the ROS
+                     service executor is unavailable. -->
+                <param name="pdo_diagnostics_auto_start">${pdo_diagnostics_auto_start}</param>
                 <param name="pdo_diagnostics_max_cycles">20000</param>
                 <param name="enable_motors_on_activate">${enable_motors_on_activate}</param>

File: src/zhishu_robot_moveit_config/config/zhishu_robot.urdf.xacro (robot description, xacro)
@@ -5,4 +5,5 @@
     <xacro:arg name="use_fake_hardware" default="true" />
     <xacro:arg name="enable_motors_on_activate" default="true" />
+    <xacro:arg name="pdo_diagnostics_auto_start" default="true" />
     <xacro:arg name="use_head_camera" default="false" />
     <xacro:arg name="hide_head_pitch_visual" default="false" />
@@ -19,10 +20,12 @@
             initial_positions_file="$(arg initial_positions_file)"
             use_fake_hardware="$(arg use_fake_hardware)"
-            enable_motors_on_activate="$(arg enable_motors_on_activate)"/>
+            enable_motors_on_activate="$(arg enable_motors_on_activate)"
+            pdo_diagnostics_auto_start="$(arg pdo_diagnostics_auto_start)"/>
         <xacro:zhishu_robot_right_arm_ros2_control
             name="RightArmSystem"
             initial_positions_file="$(arg initial_positions_file)"
             use_fake_hardware="$(arg use_fake_hardware)"
-            enable_motors_on_activate="$(arg enable_motors_on_activate)"/>
+            enable_motors_on_activate="$(arg enable_motors_on_activate)"
+            pdo_diagnostics_auto_start="$(arg pdo_diagnostics_auto_start)"/>
     </xacro:unless>
     <xacro:if value="$(arg use_gazebo)">

Commit message: feat(ethercat): 完善左臂与头腰部硬件配置
已完成仿真环境下头腰部电机控制验证，真机 EtherCAT 尚未验证。

File: src/zhishu_robot_moveit_config/config/zhishu_robot.left_arm.ros2_control.xacro (robot description, xacro)
@@ -1,5 +1,5 @@
 <?xml version="1.0"?>
 <robot xmlns:xacro="http://www.ros.org/wiki/xacro">
-    <xacro:macro name="zhishu_robot_left_arm_ros2_control" params="name initial_positions_file use_gazebo:=false use_fake_hardware:=true enable_motors_on_activate:=true pdo_diagnostics_auto_start:=true">
+    <xacro:macro name="zhishu_robot_left_arm_ros2_control" params="name initial_positions_file use_gazebo:=false use_fake_hardware:=true enable_motors_on_activate:=true pdo_diagnostics_auto_start:=true include_torso_head_state_joints:=true">
         <xacro:property name="initial_positions" value="${xacro.load_yaml(initial_positions_file)['initial_positions']}"/>
         <ros2_control name="${name}" type="system">
@@ -206,19 +206,25 @@
                 </state_interface>
             </joint>
-            <joint name="waist_pitch_joint">
-                <state_interface name="position">
-                  <param name="initial_value">${initial_positions['waist_pitch_joint']}</param>
-                </state_interface>
-            </joint>
-            <joint name="head_yaw_joint">
-                <state_interface name="position">
-                  <param name="initial_value">${initial_positions['head_yaw_joint']}</param>
-                </state_interface>
-            </joint>
-            <joint name="head_pitch_joint">
-                <state_interface name="position">
-                  <param name="initial_value">${initial_positions['head_pitch_joint']}</param>
-                </state_interface>
-            </joint>
+            <!-- Historically these three passive state interfaces lived in the
+                 left-arm component so RViz had a complete kinematic chain.
+                 Disable them when the real TorsoHeadSystem owns the joints to
+                 avoid duplicate ros2_control interfaces. -->
+            <xacro:if value="${include_torso_head_state_joints}">
+                <joint name="waist_pitch_joint">
+                    <state_interface name="position">
+                      <param name="initial_value">${initial_positions['waist_pitch_joint']}</param>
+                    </state_interface>
+                </joint>
+                <joint name="head_yaw_joint">
+                    <state_interface name="position">
+                      <param name="initial_value">${initial_positions['head_yaw_joint']}</param>
+                    </state_interface>
+                </joint>
+                <joint name="head_pitch_joint">
+                    <state_interface name="position">
+                      <param name="initial_value">${initial_positions['head_pitch_joint']}</param>
+                    </state_interface>
+                </joint>
+            </xacro:if>
             <joint name="left_wheel_joint">
                 <state_interface name="position">

File: src/zhishu_robot_moveit_config/config/zhishu_robot.urdf.xacro (robot description, xacro)
@@ -4,5 +4,9 @@
     <xacro:arg name="use_gazebo" default="false" />
     <xacro:arg name="use_fake_hardware" default="true" />
+    <xacro:arg name="enable_left_arm_hardware" default="true" />
+    <xacro:arg name="enable_right_arm_hardware" default="true" />
+    <xacro:arg name="enable_torso_head_hardware" default="false" />
     <xacro:arg name="enable_motors_on_activate" default="true" />
+    <xacro:arg name="torso_head_enable_motors_on_activate" default="false" />
     <xacro:arg name="pdo_diagnostics_auto_start" default="true" />
     <xacro:arg name="use_head_camera" default="false" />
@@ -14,18 +18,45 @@
     <xacro:include filename="zhishu_robot.left_arm.ros2_control.xacro" />
     <xacro:include filename="zhishu_robot.right_arm.ros2_control.xacro" />
+    <xacro:include filename="zhishu_robot.torso_head.ros2_control.xacro" />
     <xacro:include filename="zhishu_robot.gazebo.ros2_control.xacro" />
     <xacro:unless value="$(arg use_gazebo)">
-        <xacro:zhishu_robot_left_arm_ros2_control
-            name="LeftArmSystem"
-            initial_positions_file="$(arg initial_positions_file)"
-            use_fake_hardware="$(arg use_fake_hardware)"
-            enable_motors_on_activate="$(arg enable_motors_on_activate)"
-            pdo_diagnostics_auto_start="$(arg pdo_diagnostics_auto_start)"/>
-        <xacro:zhishu_robot_right_arm_ros2_control
-            name="RightArmSystem"
-            initial_positions_file="$(arg initial_positions_file)"
-            use_fake_hardware="$(arg use_fake_hardware)"
-            enable_motors_on_activate="$(arg enable_motors_on_activate)"
-            pdo_diagnostics_auto_start="$(arg pdo_diagnostics_auto_start)"/>
+        <xacro:if value="$(arg enable_left_arm_hardware)">
+            <!-- If TorsoHeadSystem is present it owns waist_pitch/head_yaw/head_pitch;
+                 do not export the legacy passive copies from LeftArmSystem. -->
+            <xacro:if value="$(arg enable_torso_head_hardware)">
+                <xacro:zhishu_robot_left_arm_ros2_control
+                    name="LeftArmSystem"
+                    initial_positions_file="$(arg initial_positions_file)"
+                    use_fake_hardware="$(arg use_fake_hardware)"
+                    enable_motors_on_activate="$(arg enable_motors_on_activate)"
+                    pdo_diagnostics_auto_start="$(arg pdo_diagnostics_auto_start)"
+                    include_torso_head_state_joints="false"/>
+            </xacro:if>
+            <xacro:unless value="$(arg enable_torso_head_hardware)">
+                <xacro:zhishu_robot_left_arm_ros2_control
+                    name="LeftArmSystem"
+                    initial_positions_file="$(arg initial_positions_file)"
+                    use_fake_hardware="$(arg use_fake_hardware)"
+                    enable_motors_on_activate="$(arg enable_motors_on_activate)"
+                    pdo_diagnostics_auto_start="$(arg pdo_diagnostics_auto_start)"
+                    include_torso_head_state_joints="true"/>
+            </xacro:unless>
+        </xacro:if>
+        <xacro:if value="$(arg enable_right_arm_hardware)">
+            <xacro:zhishu_robot_right_arm_ros2_control
+                name="RightArmSystem"
+                initial_positions_file="$(arg initial_positions_file)"
+                use_fake_hardware="$(arg use_fake_hardware)"
+                enable_motors_on_activate="$(arg enable_motors_on_activate)"
+                pdo_diagnostics_auto_start="$(arg pdo_diagnostics_auto_start)"/>
+        </xacro:if>
+        <xacro:if value="$(arg enable_torso_head_hardware)">
+            <xacro:zhishu_robot_torso_head_ros2_control
+                name="TorsoHeadSystem"
+                initial_positions_file="$(arg initial_positions_file)"
+                use_fake_hardware="$(arg use_fake_hardware)"
+                enable_motors_on_activate="$(arg torso_head_enable_motors_on_activate)"
+                pdo_diagnostics_auto_start="$(arg pdo_diagnostics_auto_start)"/>
+        </xacro:if>
     </xacro:unless>
     <xacro:if value="$(arg use_gazebo)">
