Commit message: fix(hardware): 合并头腰部电机到master0左臂系统

File: src/zhishu_robot_moveit_config/config/zhishu_robot.left_arm.ros2_control.xacro (robot description, xacro)
@@ -1,5 +1,5 @@
 <?xml version="1.0"?>
 <robot xmlns:xacro="http://www.ros.org/wiki/xacro">
-    <xacro:macro name="zhishu_robot_left_arm_ros2_control" params="name initial_positions_file use_gazebo:=false use_fake_hardware:=true enable_motors_on_activate:=true pdo_diagnostics_auto_start:=true include_torso_head_state_joints:=true">
+    <xacro:macro name="zhishu_robot_left_arm_ros2_control" params="name initial_positions_file use_gazebo:=false use_fake_hardware:=true enable_motors_on_activate:=true pdo_diagnostics_auto_start:=true include_torso_head_state_joints:=true include_torso_head_ethercat_joints:=false">
         <xacro:property name="initial_positions" value="${xacro.load_yaml(initial_positions_file)['initial_positions']}"/>
         <ros2_control name="${name}" type="system">
@@ -47,4 +47,8 @@
                 <param name="pdo_diagnostics_max_cycles">20000</param>
                 <param name="enable_motors_on_activate">${enable_motors_on_activate}</param>
+                <!-- Final dual-master topology:
+                     master0 = left arm (0..6) + torso/head GH1 drives (8..10).
+                     Slave 7 is the FCE1353 device shown by `ethercat slaves`, so it
+                     must remain skipped by the GH1 motor mapping. -->
                 <param name="master_index">0</param>
                 <param name="alias">0</param>
@@ -213,8 +217,51 @@
                 </state_interface>
             </joint>
-            <!-- Historically these three passive state interfaces lived in the
-                 left-arm component so RViz had a complete kinematic chain.
-                 Disable them when the real TorsoHeadSystem owns the joints to
-                 avoid duplicate ros2_control interfaces. -->
+            <!-- When torso/head shares master0 with the left arm, the same
+                 LeftEsMotorHardwareInterface instance must own all ten GH1 drives.
+                 IgH master ownership is exclusive, so do not create a second
+                 EthercatDriver for master0. The physical master0 scan currently is:
+                   0..6  = left-arm GH1
+                   7     = FCE1353 (not controlled here)
+                   8     = head yaw GH1
+                   9     = head pitch GH1
+                   10    = waist pitch GH1
+                 Positions 11..13 are FCE1353 devices and are also intentionally skipped. -->
+            <xacro:if value="${include_torso_head_ethercat_joints}">
+                <joint name="waist_pitch_joint">
+                    <param name="use_ethercat">true</param>
+                    <param name="motor_name">torso_head_motor_2</param>
+                    <param name="slave_position">10</param>
+                    <param name="reduction_ratio">101.0</param>
+                    <param name="position_wrap_reference_rad">-0.2618</param>
+                    <command_interface name="position"/>
+                    <state_interface name="position">
+                      <param name="initial_value">${initial_positions['waist_pitch_joint']}</param>
+                    </state_interface>
+                </joint>
+                <joint name="head_yaw_joint">
+                    <param name="use_ethercat">true</param>
+                    <param name="motor_name">torso_head_motor_0</param>
+                    <param name="slave_position">8</param>
+                    <param name="reduction_ratio">101.0</param>
+                    <param name="position_wrap_reference_rad">0.0</param>
+                    <command_interface name="position"/>
+                    <state_interface name="position">
+                      <param name="initial_value">${initial_positions['head_yaw_joint']}</param>
+                    </state_interface>
+                </joint>
+                <joint name="head_pitch_joint">
+                    <param name="use_ethercat">true</param>
+                    <param name="motor_name">torso_head_motor_1</param>
+                    <param name="slave_position">9</param>
+                    <param name="reduction_ratio">101.0</param>
+                    <param name="position_wrap_reference_rad">-0.0435</param>
+                    <command_interface name="position"/>
+                    <state_interface name="position">
+                      <param name="initial_value">${initial_positions['head_pitch_joint']}</param>
+                    </state_interface>
+                </joint>
+            </xacro:if>
+            <!-- Passive state-only copies are kept only when torso/head hardware
+                 is disabled, so RViz still receives a complete kinematic chain. -->
             <xacro:if value="${include_torso_head_state_joints}">
                 <joint name="waist_pitch_joint">

File: src/zhishu_robot_moveit_config/config/zhishu_robot.torso_head.ros2_control.xacro (robot description, xacro)
@@ -33,6 +33,6 @@
                 <param name="pdo_diagnostics_max_cycles">20000</param>
                 <param name="enable_motors_on_activate">${enable_motors_on_activate}</param>
-                <!-- Real-hardware test topology: torso/head drives are on IgH master 1. -->
-                <param name="master_index">1</param>
+                <!-- Final topology: torso/head share IgH master0 with the left arm. -->
+                <param name="master_index">0</param>
                 <param name="alias">0</param>
                 <param name="vendor_id">0x00206688</param>
@@ -50,11 +50,12 @@
                 <param name="joint_limit_snap_tolerance_rad">0.005</param>
             </hardware>
-            <!-- Reconstructed from real-hardware single-axis tests:
-                 slave 2 drives waist pitch, slave 1 drives head pitch, and the
-                 remaining slave 0 drives head yaw. -->
+            <!-- The original 3-axis order was head_yaw=0, head_pitch=1,
+                 waist_pitch=2. On the final master0 chain these are shifted by
+                 eight physical slaves because left-arm GH1 drives occupy 0..6
+                 and FCE1353 occupies position 7. -->
             <joint name="waist_pitch_joint">
                 <param name="use_ethercat">true</param>
                 <param name="motor_name">torso_head_motor_2</param>
-                <param name="slave_position">2</param>
+                <param name="slave_position">10</param>
                 <param name="reduction_ratio">101.0</param>
                 <param name="position_wrap_reference_rad">-0.2618</param>
@@ -67,5 +68,5 @@
                 <param name="use_ethercat">true</param>
                 <param name="motor_name">torso_head_motor_0</param>
-                <param name="slave_position">0</param>
+                <param name="slave_position">8</param>
                 <param name="reduction_ratio">101.0</param>
                 <param name="position_wrap_reference_rad">0.0</param>
@@ -78,5 +79,5 @@
                 <param name="use_ethercat">true</param>
                 <param name="motor_name">torso_head_motor_1</param>
-                <param name="slave_position">1</param>
+                <param name="slave_position">9</param>
                 <param name="reduction_ratio">101.0</param>
                 <param name="position_wrap_reference_rad">-0.0435</param>

File: src/zhishu_robot_moveit_config/config/zhishu_robot.urdf.xacro (robot description, xacro)
@@ -27,6 +27,8 @@
     <xacro:unless value="$(arg use_gazebo)">
         <xacro:if value="$(arg enable_left_arm_hardware)">
-            <!-- If TorsoHeadSystem is present it owns waist_pitch/head_yaw/head_pitch;
-                 do not export the legacy passive copies from LeftArmSystem. -->
+            <!-- master0 is owned by exactly one EthercatDriver. When torso/head
+                 hardware is enabled, merge those three GH1 axes into LeftArmSystem
+                 instead of creating a second ros2_control hardware component that
+                 would try to ecrt_request_master(0) again. -->
             <xacro:if value="$(arg enable_torso_head_hardware)">
                 <xacro:zhishu_robot_left_arm_ros2_control
@@ -36,5 +38,6 @@
                     enable_motors_on_activate="$(arg enable_motors_on_activate)"
                     pdo_diagnostics_auto_start="$(arg pdo_diagnostics_auto_start)"
-                    include_torso_head_state_joints="false"/>
+                    include_torso_head_state_joints="false"
+                    include_torso_head_ethercat_joints="true"/>
             </xacro:if>
             <xacro:unless value="$(arg enable_torso_head_hardware)">
@@ -45,5 +48,6 @@
                     enable_motors_on_activate="$(arg enable_motors_on_activate)"
                     pdo_diagnostics_auto_start="$(arg pdo_diagnostics_auto_start)"
-                    include_torso_head_state_joints="true"/>
+                    include_torso_head_state_joints="true"
+                    include_torso_head_ethercat_joints="false"/>
             </xacro:unless>
         </xacro:if>
@@ -56,11 +60,16 @@
                 pdo_diagnostics_auto_start="$(arg pdo_diagnostics_auto_start)"/>
         </xacro:if>
+        <!-- Standalone torso/head mode is still available when the left-arm
+             hardware component is disabled. In the normal combined topology,
+             LeftArmSystem already owns these three joints on master0. -->
         <xacro:if value="$(arg enable_torso_head_hardware)">
-            <xacro:zhishu_robot_torso_head_ros2_control
-                name="TorsoHeadSystem"
-                initial_positions_file="$(arg initial_positions_file)"
-                use_fake_hardware="$(arg torso_head_use_fake_hardware)"
-                enable_motors_on_activate="$(arg torso_head_enable_motors_on_activate)"
-                pdo_diagnostics_auto_start="$(arg pdo_diagnostics_auto_start)"/>
+            <xacro:unless value="$(arg enable_left_arm_hardware)">
+                <xacro:zhishu_robot_torso_head_ros2_control
+                    name="TorsoHeadSystem"
+                    initial_positions_file="$(arg initial_positions_file)"
+                    use_fake_hardware="$(arg torso_head_use_fake_hardware)"
+                    enable_motors_on_activate="$(arg torso_head_enable_motors_on_activate)"
+                    pdo_diagnostics_auto_start="$(arg pdo_diagnostics_auto_start)"/>
+            </xacro:unless>
         </xacro:if>
     </xacro:unless>
