Commit message: feat(tcp): 实现工具坐标系标定与 Gazebo 验证

File: src/zhishu_robot_moveit_config/config/zhishu_robot.urdf.xacro (robot description, xacro)
@@ -18,6 +18,21 @@
     <xacro:arg name="bottle_grasp_sim_enabled" default="false" />
     <xacro:arg name="mobile_base_sim_enabled" default="false" />
+    <!-- Simulation-only TCP pivot tool. False by default: never affects hardware bringup. -->
+    <xacro:arg name="tcp_calibration_enabled" default="false" />
+    <xacro:arg name="tcp_calibration_tool" default="probe" />
     <!-- Import zhishu_robot urdf file -->
     <xacro:include filename="$(find zhishu_robot_description)/urdf/zhishu_robot.urdf.xacro" />
+    <xacro:if value="$(arg tcp_calibration_enabled)">
+        <!-- A world-fixed fixture requires a world-fixed robot base. Keep this
+             anchor confined to TCP calibration simulation. -->
+        <link name="world"/>
+        <joint name="tcp_calibration_world_anchor" type="fixed">
+            <parent link="world"/>
+            <child link="base_footprint"/>
+            <origin xyz="0 0 0" rpy="0 0 0"/>
+        </joint>
+        <xacro:include filename="$(find zhishu_robot_tcp_calibration)/urdf/tcp_probe.xacro" />
+        <xacro:tcp_calibration_probes tool="$(arg tcp_calibration_tool)" />
+    </xacro:if>
     <!-- Import control_xacro -->
     <xacro:include filename="zhishu_robot.left_arm.ros2_control.xacro" />

Commit message: feat(workobject): 实现工件坐标系标定与 Gazebo 验证

File: src/zhishu_robot_moveit_config/config/zhishu_robot.urdf.xacro (robot description, xacro)
@@ -21,4 +21,5 @@
     <xacro:arg name="tcp_calibration_enabled" default="false" />
     <xacro:arg name="tcp_calibration_tool" default="probe" />
+    <xacro:arg name="tcp_calibration_arm" default="both" />
     <!-- Import zhishu_robot urdf file -->
     <xacro:include filename="$(find zhishu_robot_description)/urdf/zhishu_robot.urdf.xacro" />
@@ -33,5 +34,5 @@
         </joint>
         <xacro:include filename="$(find zhishu_robot_tcp_calibration)/urdf/tcp_probe.xacro" />
-        <xacro:tcp_calibration_probes tool="$(arg tcp_calibration_tool)" />
+        <xacro:tcp_calibration_probes tool="$(arg tcp_calibration_tool)" arm="$(arg tcp_calibration_arm)" />
     </xacro:if>
     <!-- Import control_xacro -->

File: src/zhishu_robot_tcp_calibration/urdf/tcp_probe.xacro (robot description, xacro)
@@ -41,5 +41,5 @@
   <!-- Both tips are rigidly fixed to the wrist/flange links.  Simulation only.
        Calibration solver DOES NOT use these fixed-tip transforms. -->
-  <xacro:macro name="tcp_calibration_probes" params="tool">
+  <xacro:macro name="tcp_calibration_probes" params="tool arm:=both">
     <xacro:if value="${tool == 'probe'}">
       <xacro:property name="left_tip_x" value="0.015"/>
@@ -64,10 +64,14 @@
       <xacro:property name="tip_yaw" value="-0.22"/>
     </xacro:if>
+    <xacro:if value="${arm == 'both' or arm == 'left'}">
     <xacro:one_probe side="left" parent="L_hand_link"
       tx="${left_tip_x}" ty="${left_tip_y}" tz="${left_tip_z}"
       rr="${tip_roll}" rp="${tip_pitch}" ry="${tip_yaw}"/>
+    </xacro:if>
+    <xacro:if value="${arm == 'both' or arm == 'right'}">
     <xacro:one_probe side="right" parent="R_hand_link"
       tx="${right_tip_x}" ty="${right_tip_y}" tz="${right_tip_z}"
       rr="${tip_roll}" rp="${tip_pitch}" ry="${tip_yaw}"/>
+    </xacro:if>
   </xacro:macro>
 </robot>
