Commit message: 初步调通MTC流程

File: src/zhishu_robot_description/urdf/gripper.xacro (robot description, xacro)
@@ -61,8 +61,8 @@
         <limit effort="1000.0" velocity="1.0" lower="-0.06" upper="0.0"/>
     </joint>
-    <link name="left_gripper_tcp"/>
-    <joint name="left_gripper_tcp_joint" type="fixed">
+    <link name="right_gripper_tcp"/>
+    <joint name="right_gripper_tcp_joint" type="fixed">
         <parent link="gripper_base_link"/>
-        <child link="left_gripper_tcp"/>
+        <child link="right_gripper_tcp"/>
         <origin xyz="0 0 0.04" rpy="1.5708 0 0"/>
     </joint>

File: src/zhishu_robot_moveit_config/config/zhishu_robot.ros2_control.xacro (robot description, xacro)
@@ -98,4 +98,34 @@
                 </state_interface>
             </joint>
+            <joint name="waist_up_down_joint">
+                <state_interface name="position">
+                  <param name="initial_value">${initial_positions['waist_up_down_joint']}</param>
+                </state_interface>
+            </joint>
+            <joint name="waist_pitch_joint">
+                <state_interface name="position">
+                  <param name="initial_value">${initial_positions['waist_pitch_joint']}</param>
+                </state_interface>
+            </joint>
+            <joint name="head_yaw_joint">
+                <state_interface name="position">
+                  <param name="initial_value">${initial_positions['head_yaw_joint']}</param>
+                </state_interface>
+            </joint>
+            <joint name="head_pitch_joint">
+                <state_interface name="position">
+                  <param name="initial_value">${initial_positions['head_pitch_joint']}</param>
+                </state_interface>
+            </joint>
+            <joint name="left_wheel_joint">
+                <state_interface name="position">
+                  <param name="initial_value">${initial_positions['left_wheel_joint']}</param>
+                </state_interface>
+            </joint>
+            <joint name="right_wheel_joint">
+                <state_interface name="position">
+                  <param name="initial_value">${initial_positions['right_wheel_joint']}</param>
+                </state_interface>
+            </joint>
         </ros2_control>
     </xacro:macro>

Commit message: 优化mtc抓取时候的方向

File: src/zhishu_robot_description/urdf/gripper.xacro (robot description, xacro)
@@ -65,5 +65,5 @@
         <parent link="gripper_base_link"/>
         <child link="right_gripper_tcp"/>
-        <origin xyz="0 0 0.04" rpy="1.5708 0 0"/>
+        <origin xyz="0 0 0.06" rpy="1.5708 0 0"/>
     </joint>
 </robot>

Commit message: 优化右臂程序

File: src/zhishu_robot_description/urdf/gripper.xacro (robot description, xacro)
@@ -11,5 +11,6 @@
         <collision>
             <geometry>
-                <box size="0.160 0.045 0.016"/>
+                <box size="0.2 0.06 0.02"/>
+                <!-- <box size="0.160 0.045 0.016"/> -->
             </geometry>
             <origin xyz="0 0 0.008" rpy="0 0 0"/>
@@ -26,5 +27,5 @@
         <collision>
             <geometry>
-                <box size="0.016 0.045 0.060"/>
+                <box size="0.02 0.06 0.08"/>
             </geometry>
             <origin xyz="0 0 0.030" rpy="0 0 0"/>
@@ -41,5 +42,5 @@
         <collision>
             <geometry>
-                <box size="0.016 0.045 0.060"/>
+                <box size="0.02 0.06 0.08"/>
             </geometry>
             <origin xyz="0 0 0.030" rpy="0 0 0"/>

File: src/zhishu_robot_description/urdf/zhishu_robot_description_dh.urdf (robot description, URDF)
Before this commit: robot zhishu_robot_description, 30 links, 29 joints
Links:
- link waist_up_down_link: geometry collision box size=0.240 0.240 0.560; visual mesh filename=package://zhishu_robot_description/meshes/waist_up_down_lin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

File: src/zhishu_robot_moveit_config/config/zhishu_robot.ros2_control.xacro (robot description, xacro)
@@ -10,5 +10,5 @@
                 <plugin>es_motor_hardware/EsMotorHardwareInterface</plugin>
                 <!-- IgH EtherCAT / GH1 SERVOPACK defaults. Per-joint params below can override these. -->
-                <param name="cycle_ns">1000000</param>
+                <param name="cycle_ns">2000000</param>
                 <param name="enable_dc">true</param>
                 <param name="assign_activate">0x0300</param>
