Commit message: 左工具也改成夹爪

File: src/zhishu_robot_description/urdf/gripper.xacro (robot description, xacro)
@@ -12,5 +12,4 @@
             <geometry>
                 <box size="0.2 0.06 0.02"/>
-                <!-- <box size="0.160 0.045 0.016"/> -->
             </geometry>
             <origin xyz="0 0 0.008" rpy="0 0 0"/>
@@ -68,3 +67,70 @@
         <origin xyz="0 0 0.06" rpy="1.5708 0 0"/>
     </joint>
+    <!-- Left gripper: same geometry and kinematics as the right gripper, but with left_* names. -->
+    <link name="left_gripper_base_link">
+        <visual>
+            <geometry>
+                <box size="0.2 0.06 0.02"/>
+            </geometry>
+            <origin xyz="0 0 0.01" rpy="0 0 0"/>
+            <material name="dark_green"/>
+        </visual>
+        <collision>
+            <geometry>
+                <box size="0.2 0.06 0.02"/>
+            </geometry>
+            <origin xyz="0 0 0.008" rpy="0 0 0"/>
+        </collision>
+    </link>
+    <link name="left_gripper_left_finger_link">
+        <visual>
+            <geometry>
+                <box size="0.02 0.06 0.08"/>
+            </geometry>
+            <origin xyz="0 0 0.04" rpy="0 0 0"/>
+            <material name="light_green"/>
+        </visual>
+        <collision>
+            <geometry>
+                <box size="0.02 0.06 0.08"/>
+            </geometry>
+            <origin xyz="0 0 0.030" rpy="0 0 0"/>
+        </collision>
+    </link>
+    <link name="left_gripper_right_finger_link">
+        <visual>
+            <geometry>
+                <box size="0.02 0.06 0.08"/>
+            </geometry>
+            <origin xyz="0 0 0.04" rpy="0 0 0"/>
+            <material name="light_green"/>
+        </visual>
+        <collision>
+            <geometry>
+                <box size="0.02 0.06 0.08"/>
+            </geometry>
+            <origin xyz="0 0 0.030" rpy="0 0 0"/>
+        </collision>
+    </link>
+    <joint name="left_gripper_left_finger_joint" type="prismatic">
+        <parent link="left_gripper_base_link"/>
+        <child link="left_gripper_left_finger_link"/>
+        <origin xyz="-0.07 0 0.02" rpy="0 0 0"/>
+        <axis xyz="1 0 0"/>
+        <limit effort="1000.0" velocity="1.0" lower="0.0" upper="0.06"/>
+    </joint>
+    <joint name="left_gripper_right_finger_joint" type="prismatic">
+        <parent link="left_gripper_base_link"/>
+        <child link="left_gripper_right_finger_link"/>
+        <origin xyz="0.07 0 0.02" rpy="0 0 0"/>
+        <axis xyz="1 0 0"/>
+        <mimic joint="left_gripper_left_finger_joint" multiplier="-1.0"/>
+        <limit effort="1000.0" velocity="1.0" lower="-0.06" upper="0.0"/>
+    </joint>
+    <link name="left_gripper_tcp"/>
+    <joint name="left_gripper_tcp_joint" type="fixed">
+        <parent link="left_gripper_base_link"/>
+        <child link="left_gripper_tcp"/>
+        <origin xyz="0 0 0.06" rpy="1.5708 0 0"/>
+    </joint>
 </robot>

File: src/zhishu_robot_description/urdf/zhishu_robot.gazebo.urdf.xacro (robot description, xacro)
@@ -4,4 +4,9 @@
     <xacro:include filename="$(find zhishu_robot_description)/urdf/gripper.xacro"/>
     <xacro:include filename="$(find zhishu_robot_description)/urdf/zhishu_robot_description_dh.urdf"/>
+    <joint name="left_gripper_joint" type="fixed">
+        <parent link="L_hand_link" />
+        <child link="left_gripper_base_link" />
+        <origin xyz="0 0 0" rpy="0 3.14159 0" />
+    </joint>
     <joint name="right_gripper_joint" type="fixed">
         <parent link="R_hand_link" />

File: src/zhishu_robot_description/urdf/zhishu_robot.urdf.xacro (robot description, xacro)
@@ -4,4 +4,9 @@
     <xacro:include filename="$(find zhishu_robot_description)/urdf/gripper.xacro"/>
     <xacro:include filename="$(find zhishu_robot_description)/urdf/zhishu_robot_description_dh.urdf"/>
+    <joint name="left_gripper_joint" type="fixed">
+        <parent link="L_hand_link" />
+        <child link="left_gripper_base_link" />
+        <origin xyz="0 0 0" rpy="0 3.14159 0" />
+    </joint>
     <joint name="right_gripper_joint" type="fixed">
         <parent link="R_hand_link" />

File: src/zhishu_robot_description/urdf/zhishu_robot_description_dh.urdf (robot description, URDF)
Before this commit: robot zhishu_robot_description, 30 links, 29 joints
Links:
- link L_hand_link: mass 0.079329 -> None; geometry 

File: src/zhishu_robot_moveit_config/config/zhishu_robot.left_arm.ros2_control.xacro (robot description, xacro)
@@ -99,4 +99,14 @@
                 </state_interface>
             </joint>
+            <joint name="left_gripper_left_finger_joint">
+                <command_interface name="position"/>
+                <state_interface name="position">
+                  <param name="initial_value">${initial_positions['left_gripper_left_finger_joint']}</param>
+                </state_interface>
+            </joint>
+            <!-- Keep both non-EtherCAT gripper command interfaces in one mock
+                 hardware component. GenericSystem on ROS 2 Humble receives the
+                 complete mode-switch request and rejects foreign gripper joints
+                 when the two grippers are split across different components. -->
             <joint name="gripper_left_finger_joint">
                 <command_interface name="position"/>

File: src/zhishu_robot_moveit_config/config/zhishu_robot.right_arm.ros2_control.xacro (robot description, xacro)
@@ -99,11 +99,5 @@
                 </state_interface>
             </joint>
-            <!-- <joint name="gripper_left_finger_joint">
-                <command_interface name="position"/>
-                <state_interface name="position">
-                  <param name="initial_value">${initial_positions['gripper_left_finger_joint']}</param>
-                </state_interface>
-            </joint>
-            <joint name="waist_up_down_joint">
+            <!-- <joint name="waist_up_down_joint">
                 <state_interface name="position">
                   <param name="initial_value">${initial_positions['waist_up_down_joint']}</param>

Commit message: 增加双手搬运物料箱子demo

File: src/zhishu_robot_description/urdf/gripper.xacro (robot description, xacro)
@@ -65,5 +65,5 @@
         <parent link="gripper_base_link"/>
         <child link="right_gripper_tcp"/>
-        <origin xyz="0 0 0.06" rpy="1.5708 0 0"/>
+        <origin xyz="0 0 0.10" rpy="1.5708 0 0"/>
     </joint>
     <!-- Left gripper: same geometry and kinematics as the right gripper, but with left_* names. -->
@@ -132,5 +132,5 @@
         <parent link="left_gripper_base_link"/>
         <child link="left_gripper_tcp"/>
-        <origin xyz="0 0 0.06" rpy="1.5708 0 0"/>
+        <origin xyz="0 0 0.10" rpy="1.5708 0 0"/>
     </joint>
 </robot>

Commit message: 夹爪高度改成0.2

File: src/zhishu_robot_description/urdf/gripper.xacro (robot description, xacro)
@@ -19,14 +19,14 @@
         <visual>
             <geometry>
-                <box size="0.02 0.06 0.08"/>
+                <box size="0.02 0.06 0.20"/>
             </geometry>
-            <origin xyz="0 0 0.04" rpy="0 0 0"/>
+            <origin xyz="0 0 0.10" rpy="0 0 0"/>
             <material name="light_green"/>
         </visual>
         <collision>
             <geometry>
-                <box size="0.02 0.06 0.08"/>
+                <box size="0.02 0.06 0.20"/>
             </geometry>
-            <origin xyz="0 0 0.030" rpy="0 0 0"/>
+            <origin xyz="0 0 0.10" rpy="0 0 0"/>
         </collision>
     </link>
@@ -34,14 +34,14 @@
         <visual>
             <geometry>
-                <box size="0.02 0.06 0.08"/>
+                <box size="0.02 0.06 0.20"/>
             </geometry>
-            <origin xyz="0 0 0.04" rpy="0 0 0"/>
+            <origin xyz="0 0 0.10" rpy="0 0 0"/>
             <material name="light_green"/>
         </visual>
         <collision>
             <geometry>
-                <box size="0.02 0.06 0.08"/>
+                <box size="0.02 0.06 0.20"/>
             </geometry>
-            <origin xyz="0 0 0.030" rpy="0 0 0"/>
+            <origin xyz="0 0 0.10" rpy="0 0 0"/>
         </collision>
     </link>
@@ -65,5 +65,5 @@
         <parent link="gripper_base_link"/>
         <child link="right_gripper_tcp"/>
-        <origin xyz="0 0 0.10" rpy="1.5708 0 0"/>
+        <origin xyz="0 0 0.12" rpy="1.5708 0 0"/>
     </joint>
     <!-- Left gripper: same geometry and kinematics as the right gripper, but with left_* names. -->
@@ -86,14 +86,14 @@
         <visual>
             <geometry>
-                <box size="0.02 0.06 0.08"/>
+                <box size="0.02 0.06 0.20"/>
             </geometry>
-            <origin xyz="0 0 0.04" rpy="0 0 0"/>
+            <origin xyz="0 0 0.10" rpy="0 0 0"/>
             <material name="light_green"/>
         </visual>
         <collision>
             <geometry>
-                <box size="0.02 0.06 0.08"/>
+                <box size="0.02 0.06 0.20"/>
             </geometry>
-            <origin xyz="0 0 0.030" rpy="0 0 0"/>
+            <origin xyz="0 0 0.10" rpy="0 0 0"/>
         </collision>
     </link>
@@ -101,14 +101,14 @@
         <visual>
             <geometry>
-                <box size="0.02 0.06 0.08"/>
+                <box size="0.02 0.06 0.20"/>
             </geometry>
-            <origin xyz="0 0 0.04" rpy="0 0 0"/>
+            <origin xyz="0 0 0.10" rpy="0 0 0"/>
             <material name="light_green"/>
         </visual>
         <collision>
             <geometry>
-                <box size="0.02 0.06 0.08"/>
+                <box size="0.02 0.06 0.20"/>
             </geometry>
-            <origin xyz="0 0 0.030" rpy="0 0 0"/>
+            <origin xyz="0 0 0.10" rpy="0 0 0"/>
         </collision>
     </link>
@@ -132,5 +132,5 @@
         <parent link="left_gripper_base_link"/>
         <child link="left_gripper_tcp"/>
-        <origin xyz="0 0 0.10" rpy="1.5708 0 0"/>
+        <origin xyz="0 0 0.12" rpy="1.5708 0 0"/>
     </joint>
 </robot>

File: src/zhishu_robot_description/urdf/zhishu_robot_description_dh.urdf (robot description, URDF)
Before this commit: robot zhishu_robot_description, 30 links, 29 joints
Links:
- link base_link: geometry collision box size=0.450 0.350 0.300; visual mesh filename=package://zhishu_robot_description/meshes/base_link.STL

Commit message: crate carry增加一个起始位置过渡点

File: src/zhishu_robot_description/urdf/gripper.xacro (robot description, xacro)
@@ -65,5 +65,5 @@
         <parent link="gripper_base_link"/>
         <child link="right_gripper_tcp"/>
-        <origin xyz="0 0 0.12" rpy="1.5708 0 0"/>
+        <origin xyz="0 0 0.18" rpy="1.5708 0 0"/>
     </joint>
     <!-- Left gripper: same geometry and kinematics as the right gripper, but with left_* names. -->
@@ -132,5 +132,5 @@
         <parent link="left_gripper_base_link"/>
         <child link="left_gripper_tcp"/>
-        <origin xyz="0 0 0.12" rpy="1.5708 0 0"/>
+        <origin xyz="0 0 0.18" rpy="1.5708 0 0"/>
     </joint>
 </robot>

Commit message: feat(handeye): 支持法兰直装 ChArUco 标定板仿真

File: src/zhishu_robot_description/urdf/gripper.xacro (robot description, xacro)
@@ -84,49 +84,58 @@
     <!-- Left gripper: same geometry and kinematics as the right gripper, but with left_* names. -->
     <link name="left_gripper_base_link">
-        <visual>
-            <geometry>
-                <box size="0.2 0.06 0.02"/>
-            </geometry>
-            <origin xyz="0 0 0.01" rpy="0 0 0"/>
-            <material name="dark_green"/>
-        </visual>
-        <collision>
-            <geometry>
-                <box size="0.2 0.06 0.02"/>
-            </geometry>
-            <origin xyz="0 0 0.008" rpy="0 0 0"/>
-        </collision>
+        <!-- Keep the logical gripper joints in hand-eye mode so the shared
+             SRDF and ros2_control configuration remain valid, but remove the
+             physical tool from both rendering and collision checking. -->
+        <xacro:unless value="$(arg handeye_target_enabled)">
+            <visual>
+                <geometry>
+                    <box size="0.2 0.06 0.02"/>
+                </geometry>
+                <origin xyz="0 0 0.01" rpy="0 0 0"/>
+                <material name="dark_green"/>
+            </visual>
+            <collision>
+                <geometry>
+                    <box size="0.2 0.06 0.02"/>
+                </geometry>
+                <origin xyz="0 0 0.008" rpy="0 0 0"/>
+            </collision>
+        </xacro:unless>
     </link>
     <link name="left_gripper_left_finger_link">
         <xacro:gripper_finger_inertial/>
-        <visual>
-            <geometry>
-                <box size="0.02 0.06 0.20"/>
-            </geometry>
-            <origin xyz="0 0 0.10" rpy="0 0 0"/>
-            <material name="light_green"/>
-        </visual>
-        <collision>
-            <geometry>
-                <box size="0.02 0.06 0.20"/>
-            </geometry>
-            <origin xyz="0 0 0.10" rpy="0 0 0"/>
-        </collision>
+        <xacro:unless value="$(arg handeye_target_enabled)">
+            <visual>
+                <geometry>
+                    <box size="0.02 0.06 0.20"/>
+                </geometry>
+                <origin xyz="0 0 0.10" rpy="0 0 0"/>
+                <material name="light_green"/>
+            </visual>
+            <collision>
+                <geometry>
+                    <box size="0.02 0.06 0.20"/>
+                </geometry>
+                <origin xyz="0 0 0.10" rpy="0 0 0"/>
+            </collision>
+        </xacro:unless>
     </link>
     <link name="left_gripper_right_finger_link">
         <xacro:gripper_finger_inertial/>
-        <visual>
-            <geometry>
-                <box size="0.02 0.06 0.20"/>
-            </geometry>
-            <origin xyz="0 0 0.10" rpy="0 0 0"/>
-            <material name="light_green"/>
-        </visual>
-        <collision>
-            <geometry>
-                <box size="0.02 0.06 0.20"/>
-            </geometry>
-            <origin xyz="0 0 0.10" rpy="0 0 0"/>
-        </collision>
+        <xacro:unless value="$(arg handeye_target_enabled)">
+            <visual>
+                <geometry>
+                    <box size="0.02 0.06 0.20"/>
+                </geometry>
+                <origin xyz="0 0 0.10" rpy="0 0 0"/>
+                <material name="light_green"/>
+            </visual>
+            <collision>
+                <geometry>
+                    <box size="0.02 0.06 0.20"/>
+                </geometry>
+                <origin xyz="0 0 0.10" rpy="0 0 0"/>
+            </collision>
+        </xacro:unless>
     </link>
     <joint name="left_gripper_left_finger_joint" type="prismatic">

File: src/zhishu_robot_description/urdf/handeye_target_pattern.xacro (robot description, xacro)
@@ -3,8 +3,10 @@
   <!-- Generated 7x5 DICT_4X4_50 ChArUco board:
        square_length=0.030 m, marker_length=0.022 m.
+       The photo-estimated carrier plate is 0.240 x 0.220 x 0.003 m.
        The pattern is mirrored onto local -X because that is the camera-facing side. -->
   <xacro:macro name="handeye_target_pattern">
     <visual name="handeye_board_backing">
-      <geometry><box size="0.003 0.2300000 0.1700000"/></geometry>
+      <origin xyz="0 0 -0.0200000" rpy="0 0 0"/>
+      <geometry><box size="0.0030000 0.2400000 0.2200000"/></geometry>
       <material name="handeye_white"><color rgba="1 1 1 1"/></material>
     </visual>

File: src/zhishu_robot_description/urdf/head_camera_handeye.xacro (robot description, xacro)
@@ -56,18 +56,57 @@
     </xacro:if>
   </xacro:macro>
-  <!-- Calibration target is visual-only and fixed to the left TCP.  It is
-       named *_truth so the detector can publish handeye_target independently. -->
+  <!-- The physical calibration plate replaces the left gripper only while
+       hand-eye mode is enabled.  Dimensions and hole locations below are
+       estimated from the supplied photograph after rectifying it against the
+       known 30 mm ChArUco squares.  The ChArUco pattern frame remains at the
+       pattern center, with local -X as the printed/camera-facing side. -->
   <xacro:macro name="left_handeye_target" params="enabled">
     <xacro:if value="${enabled}">
       <link name="handeye_target_truth">
-        <!-- The board's local normal is +X. The generated macro uses colored
-             box geometry instead of a texture for headless OGRE compatibility. -->
+        <inertial>
+          <origin xyz="0 0 -0.020" rpy="0 0 0"/>
+          <mass value="0.43"/>
+          <inertia ixx="0.0037983" ixy="0" ixz="0"
+                   iyy="0.0017347" iyz="0" izz="0.0020643"/>
+        </inertial>
+        <collision>
+          <origin xyz="0 0 -0.020" rpy="0 0 0"/>
+          <geometry><box size="0.003 0.240 0.220"/></geometry>
+        </collision>
+        <!-- Generated box geometry is used instead of a texture so the
+             detector also works with the headless OGRE renderer. -->
         <xacro:handeye_target_pattern/>
+        <!-- Photo-estimated 5.5 mm flange holes.  URDF has no subtraction
+             primitive, so these thin dark discs are visual alignment marks;
+             the collision model remains one conservative plate box. -->
+        <visual name="handeye_mount_hole_1">
+          <origin xyz="-0.0017 -0.0207 -0.0912" rpy="0 ${pi / 2} 0"/>
+          <geometry><cylinder radius="0.00275" length="0.0004"/></geometry>
+          <material name="handeye_hole"><color rgba="0.35 0.35 0.35 1"/></material>
+        </visual>
+        <visual name="handeye_mount_hole_2">
+          <origin xyz="-0.0017 -0.0206 -0.1226" rpy="0 ${pi / 2} 0"/>
+          <geometry><cylinder radius="0.00275" length="0.0004"/></geometry>
+          <material name="handeye_hole"><color rgba="0.35 0.35 0.35 1"/></material>
+        </visual>
+        <visual name="handeye_mount_hole_3">
+          <origin xyz="-0.0017 0.0213 -0.0985" rpy="0 ${pi / 2} 0"/>
+          <geometry><cylinder radius="0.00275" length="0.0004"/></geometry>
+          <material name="handeye_hole"><color rgba="0.35 0.35 0.35 1"/></material>
+        </visual>
+        <visual name="handeye_mount_hole_4">
+          <origin xyz="-0.0017 0.0214 -0.1152" rpy="0 ${pi / 2} 0"/>
+          <geometry><cylinder radius="0.00275" length="0.0004"/></geometry>
+          <material name="handeye_hole"><color rgba="0.35 0.35 0.35 1"/></material>
+        </visual>
       </link>
       <joint name="handeye_target_mount_joint" type="fixed">
-        <parent link="left_gripper_tcp"/>
+        <parent link="L_hand_link"/>
         <child link="handeye_target_truth"/>
-        <!-- Simulated bracket keeps the board clear of the forearm silhouette. -->
-        <origin xyz="0.25 0.15 0" rpy="0 0 0"/>
+        <!-- The four-hole centroid is aligned with the flange origin.  The
+             L_hand_link mesh extends into -Z, so its free flange side is +Z.
+             The plate back (+X) touches z=0 and the printed face (-X) points
+             outward along L_hand_link +Z toward the head camera. -->
+        <origin xyz="0.1069 -0.0004 0.0015" rpy="0 ${pi / 2} 0"/>
       </joint>
     </xacro:if>

File: src/zhishu_robot_description/urdf/zhishu_robot.gazebo.urdf.xacro (robot description, xacro)
@@ -1,4 +1,5 @@
 <?xml version="1.0"?>
 <robot name="zhishu_robot" xmlns:xacro="http://www.ros.org/wiki/xacro">
+    <xacro:arg name="handeye_target_enabled" default="false"/>
     <xacro:include filename="$(find zhishu_robot_description)/urdf/common_properties.xacro"/>
     <xacro:include filename="$(find zhishu_robot_description)/urdf/gripper.xacro"/>
