Commit message: feat(grasp): 增加15kg托盘料箱预抽出与双臂转运仿真

File: src/zhishu_robot_description/urdf/gripper.xacro (robot description, xacro)
@@ -6,10 +6,12 @@
     <xacro:macro name="gripper_finger_inertial">
         <inertial>
-            <origin xyz="0 0 0.10" rpy="0 0 0"/>
+            <!-- 275 mm fingers reach the lower edge of the tote handle when
+                 the TCP stays in the arm's reachable upper hook pose. -->
+            <origin xyz="0 0 0.1375" rpy="0 0 0"/>
             <mass value="0.1"/>
             <inertia
-                ixx="0.000363333" ixy="0.0" ixz="0.0"
-                iyy="0.000336667" iyz="0.0"
-                izz="0.000033333"/>
+                ixx="0.000660208" ixy="0.0" ixz="0.0"
+                iyy="0.000631042" iyz="0.0"
+                izz="0.000036667"/>
         </inertial>
     </xacro:macro>
@@ -33,14 +35,14 @@
         <visual>
             <geometry>
-                <box size="0.02 0.06 0.20"/>
+                <box size="0.02 0.06 0.275"/>
             </geometry>
-            <origin xyz="0 0 0.10" rpy="0 0 0"/>
+            <origin xyz="0 0 0.1375" rpy="0 0 0"/>
             <material name="light_green"/>
         </visual>
         <collision>
             <geometry>
-                <box size="0.02 0.06 0.20"/>
+                <box size="0.02 0.06 0.275"/>
             </geometry>
-            <origin xyz="0 0 0.10" rpy="0 0 0"/>
+            <origin xyz="0 0 0.1375" rpy="0 0 0"/>
         </collision>
     </link>
@@ -49,14 +51,32 @@
         <visual>
             <geometry>
-                <box size="0.02 0.06 0.20"/>
+                <box size="0.02 0.06 0.275"/>
             </geometry>
-            <origin xyz="0 0 0.10" rpy="0 0 0"/>
+            <origin xyz="0 0 0.1375" rpy="0 0 0"/>
             <material name="light_green"/>
         </visual>
         <collision>
             <geometry>
-                <box size="0.02 0.06 0.20"/>
+                <box size="0.02 0.06 0.275"/>
             </geometry>
-            <origin xyz="0 0 0.10" rpy="0 0 0"/>
+            <origin xyz="0 0 0.1375" rpy="0 0 0"/>
+        </collision>
+        <!-- Broad low hook pad on the inner/right finger.  The vertical finger
+             reaches the aperture's lower edge; this pad provides a positive
+             bearing surface behind the real handle rail during the pull. -->
+        <visual>
+            <geometry>
+                <box size="0.06 0.12 0.02"/>
+            </geometry>
+            <!-- Shift inward from the right finger's +X joint offset so the
+                 pad actually overlaps the tote's 120 mm handle rail. -->
+            <origin xyz="-0.115 -0.04 0.238" rpy="0 0 0"/>
+            <material name="light_green"/>
+        </visual>
+        <collision>
+            <geometry>
+                <box size="0.06 0.12 0.02"/>
+            </geometry>
+            <origin xyz="-0.115 -0.04 0.238" rpy="0 0 0"/>
         </collision>
     </link>
@@ -66,5 +86,8 @@
         <origin xyz="-0.07 0 0.02" rpy="0 0 0"/>
         <axis xyz="1 0 0"/>
-        <limit effort="1000.0" velocity="1.0" lower="0.0" upper="0.06"/>
+        <!-- Allow a small state-estimation/controller settling margin around
+             the physical 60 mm stroke; the close command still targets the
+             real 0..60 mm range. -->
+        <limit effort="1000.0" velocity="1.0" lower="-0.01" upper="0.07"/>
     </joint>
     <joint name="gripper_right_finger_joint" type="prismatic">
@@ -74,5 +97,5 @@
         <axis xyz="1 0 0"/>
         <mimic joint="gripper_left_finger_joint" multiplier="-1.0"/>
-        <limit effort="1000.0" velocity="1.0" lower="-0.06" upper="0.0"/>
+        <limit effort="1000.0" velocity="1.0" lower="-0.07" upper="0.01"/>
     </joint>
     <link name="right_gripper_tcp"/>
@@ -108,14 +131,14 @@
             <visual>
                 <geometry>
-                    <box size="0.02 0.06 0.20"/>
+                    <box size="0.02 0.06 0.275"/>
                 </geometry>
-                <origin xyz="0 0 0.10" rpy="0 0 0"/>
+                <origin xyz="0 0 0.1375" rpy="0 0 0"/>
                 <material name="light_green"/>
             </visual>
             <collision>
                 <geometry>
-                    <box size="0.02 0.06 0.20"/>
+                    <box size="0.02 0.06 0.275"/>
                 </geometry>
-                <origin xyz="0 0 0.10" rpy="0 0 0"/>
+                <origin xyz="0 0 0.1375" rpy="0 0 0"/>
             </collision>
         </xacro:unless>
@@ -126,14 +149,14 @@
             <visual>
                 <geometry>
-                    <box size="0.02 0.06 0.20"/>
+                    <box size="0.02 0.06 0.275"/>
                 </geometry>
-                <origin xyz="0 0 0.10" rpy="0 0 0"/>
+                <origin xyz="0 0 0.1375" rpy="0 0 0"/>
                 <material name="light_green"/>
             </visual>
             <collision>
                 <geometry>
-                    <box size="0.02 0.06 0.20"/>
+                    <box size="0.02 0.06 0.275"/>
                 </geometry>
-                <origin xyz="0 0 0.10" rpy="0 0 0"/>
+                <origin xyz="0 0 0.1375" rpy="0 0 0"/>
             </collision>
         </xacro:unless>
@@ -144,5 +167,5 @@
         <origin xyz="-0.07 0 0.02" rpy="0 0 0"/>
         <axis xyz="1 0 0"/>
-        <limit effort="1000.0" velocity="1.0" lower="0.0" upper="0.06"/>
+        <limit effort="1000.0" velocity="1.0" lower="-0.01" upper="0.07"/>
     </joint>
     <joint name="left_gripper_right_finger_joint" type="prismatic">
@@ -152,5 +175,5 @@
         <axis xyz="1 0 0"/>
         <mimic joint="left_gripper_left_finger_joint" multiplier="-1.0"/>
-        <limit effort="1000.0" velocity="1.0" lower="-0.06" upper="0.0"/>
+        <limit effort="1000.0" velocity="1.0" lower="-0.07" upper="0.01"/>
     </joint>
     <link name="left_gripper_tcp"/>

File: src/zhishu_robot_moveit_config/config/zhishu_robot.urdf.xacro (robot description, xacro)
@@ -17,4 +17,5 @@
     <xacro:arg name="handeye_target_enabled" default="false" />
     <xacro:arg name="bottle_grasp_sim_enabled" default="false" />
+    <xacro:arg name="mobile_base_sim_enabled" default="false" />
     <!-- Import zhishu_robot urdf file -->
     <xacro:include filename="$(find zhishu_robot_description)/urdf/zhishu_robot.urdf.xacro" />
@@ -76,4 +77,36 @@
                 <position_proportional_gain>1.0</position_proportional_gain>
             </plugin>
+            <xacro:if value="$(arg mobile_base_sim_enabled)">
+                <!-- Simulation-only mobile base. The wheel joints are state-only in
+                     gz_ros2_control, so DiffDrive is the sole wheel command writer. -->
+                <plugin filename="gz-sim-diff-drive-system" name="gz::sim::systems::DiffDrive">
+                    <left_joint>left_wheel_joint</left_joint>
+                    <right_joint>right_wheel_joint</right_joint>
+                    <wheel_separation>0.35</wheel_separation>
+                    <wheel_radius>0.0858</wheel_radius>
+                    <topic>/cmd_vel</topic>
+                    <odom_topic>/odom</odom_topic>
+                    <tf_topic>/tf</tf_topic>
+                    <frame_id>odom</frame_id>
+                    <child_frame_id>base_footprint</child_frame_id>
+                    <odom_publish_frequency>50</odom_publish_frequency>
+                </plugin>
+            </xacro:if>
+            <!-- Extraction runs start already aligned with r0_c0.  Add
+                 wheel damping/contact friction so arm reaction forces do not
+                 roll the chassis away from the 20 cm station while the hook
+                 trajectory is executing. -->
+            <gazebo reference="left_wheel_link">
+                <mu1>8.0</mu1>
+                <mu2>8.0</mu2>
+                <kp>1000000.0</kp>
+                <kd>100.0</kd>
+            </gazebo>
+            <gazebo reference="right_wheel_link">
+                <mu1>8.0</mu1>
+                <mu2>8.0</mu2>
+                <kp>1000000.0</kp>
+                <kd>100.0</kd>
+            </gazebo>
             <xacro:if value="$(arg bottle_grasp_sim_enabled)">
                 <!-- Contact determines closure timing; this simulation-only
