Commit message: fix(grasp): 优化148mm料箱浅夹取与稳定转运（200mm夹爪，弯腰下限-90°，实际最大弯腰约-63.03°）
本提交对应200mm手指、140mm TCP固定偏移方案。
腰部允许下限为-90°；独立完整仿真遥测实际最小角度为-63.02537°，约-63.03°。
动作目标：初始停车-17.19°，预抽出-57.30°，准备直腰0°，双臂抓取/后撤-63.03°，携带-5.73°，桌边入箱/撤爪/最终停车-11.46°。
实际最大角度依据pallet_bin_video_20261007_final148/telemetry.jsonl；目标角度不等同于瞬时实测值。
不包含随后360mm夹爪、最大弯腰-45°候选方案。

File: src/zhishu_robot_description/urdf/gripper.xacro (robot description, xacro)
@@ -1,4 +1,5 @@
 <?xml version='1.0' encoding='UTF-8'?>
 <robot xmlns:xacro="http://www.ros.org/wiki/xacro">
+    <xacro:property name="tote_finger_length" value="0.200"/>
     <!-- Gazebo Sim only creates dynamic links that have valid inertial data.
          Without this block the finger links, their prismatic joints, and the
@@ -6,11 +7,11 @@
     <xacro:macro name="gripper_finger_inertial">
         <inertial>
-            <!-- 275 mm fingers reach the lower edge of the tote handle when
-                 the TCP stays in the arm's reachable upper hook pose. -->
-            <origin xyz="0 0 0.1375" rpy="0 0 0"/>
+            <!-- Candidate 200 mm fingers; TCP is 80 mm behind the tip.
+                 The tote grasp target limits insertion to about 50 mm. -->
+            <origin xyz="0 0 ${tote_finger_length / 2}" rpy="0 0 0"/>
             <mass value="0.1"/>
             <inertia
-                ixx="0.000660208" ixy="0.0" ixz="0.0"
-                iyy="0.000631042" iyz="0.0"
+                ixx="${0.1 * (0.06**2 + tote_finger_length**2) / 12}" ixy="0.0" ixz="0.0"
+                iyy="${0.1 * (0.02**2 + tote_finger_length**2) / 12}" iyz="0.0"
                 izz="0.000036667"/>
         </inertial>
@@ -35,14 +36,14 @@
         <visual>
             <geometry>
-                <box size="0.02 0.06 0.275"/>
+                <box size="0.02 0.06 ${tote_finger_length}"/>
             </geometry>
-            <origin xyz="0 0 0.1375" rpy="0 0 0"/>
+            <origin xyz="0 0 ${tote_finger_length / 2}" rpy="0 0 0"/>
             <material name="light_green"/>
         </visual>
         <collision>
             <geometry>
-                <box size="0.02 0.06 0.275"/>
+                <box size="0.02 0.06 ${tote_finger_length}"/>
             </geometry>
-            <origin xyz="0 0 0.1375" rpy="0 0 0"/>
+            <origin xyz="0 0 ${tote_finger_length / 2}" rpy="0 0 0"/>
         </collision>
     </link>
@@ -51,33 +52,18 @@
         <visual>
             <geometry>
-                <box size="0.02 0.06 0.275"/>
+                <box size="0.02 0.06 ${tote_finger_length}"/>
             </geometry>
-            <origin xyz="0 0 0.1375" rpy="0 0 0"/>
+            <origin xyz="0 0 ${tote_finger_length / 2}" rpy="0 0 0"/>
             <material name="light_green"/>
         </visual>
         <collision>
             <geometry>
-                <box size="0.02 0.06 0.275"/>
+                <box size="0.02 0.06 ${tote_finger_length}"/>
             </geometry>
-            <origin xyz="0 0 0.1375" rpy="0 0 0"/>
+            <origin xyz="0 0 ${tote_finger_length / 2}" rpy="0 0 0"/>
         </collision>
-        <!-- Broad low hook pad on the inner/right finger.  The vertical finger
-             reaches the aperture's lower edge; this pad provides a positive
-             bearing surface behind the real handle rail during the pull. -->
-        <visual>
-            <geometry>
-                <box size="0.06 0.12 0.02"/>
-            </geometry>
-            <!-- Shift inward from the right finger's +X joint offset so the
-                 pad actually overlaps the tote's 120 mm handle rail. -->
-            <origin xyz="-0.115 -0.04 0.238" rpy="0 0 0"/>
-            <material name="light_green"/>
-        </visual>
-        <collision>
-            <geometry>
-                <box size="0.06 0.12 0.02"/>
-            </geometry>
-            <origin xyz="-0.115 -0.04 0.238" rpy="0 0 0"/>
-        </collision>
+        <!-- No auxiliary crossbar/pad: the two long fingers clamp the
+             continuous tote wall directly.  The former 60x120x20 mm pad
+             could overlap the mobile-base shell at the 20 cm dock. -->
     </link>
     <joint name="gripper_left_finger_joint" type="prismatic">
@@ -103,5 +89,5 @@
         <parent link="gripper_base_link"/>
         <child link="right_gripper_tcp"/>
-        <origin xyz="0 0 0.18" rpy="1.5708 0 0"/>
+        <origin xyz="0 0 0.14" rpy="1.5708 0 0"/>
     </joint>
     <!-- Left gripper: same geometry and kinematics as the right gripper, but with left_* names. -->
@@ -131,14 +117,14 @@
             <visual>
                 <geometry>
-                    <box size="0.02 0.06 0.275"/>
+                    <box size="0.02 0.06 ${tote_finger_length}"/>
                 </geometry>
-                <origin xyz="0 0 0.1375" rpy="0 0 0"/>
+                <origin xyz="0 0 ${tote_finger_length / 2}" rpy="0 0 0"/>
                 <material name="light_green"/>
             </visual>
             <collision>
                 <geometry>
-                    <box size="0.02 0.06 0.275"/>
+                    <box size="0.02 0.06 ${tote_finger_length}"/>
                 </geometry>
-                <origin xyz="0 0 0.1375" rpy="0 0 0"/>
+                <origin xyz="0 0 ${tote_finger_length / 2}" rpy="0 0 0"/>
             </collision>
         </xacro:unless>
@@ -149,14 +135,14 @@
             <visual>
                 <geometry>
-                    <box size="0.02 0.06 0.275"/>
+                    <box size="0.02 0.06 ${tote_finger_length}"/>
                 </geometry>
-                <origin xyz="0 0 0.1375" rpy="0 0 0"/>
+                <origin xyz="0 0 ${tote_finger_length / 2}" rpy="0 0 0"/>
                 <material name="light_green"/>
             </visual>
             <collision>
                 <geometry>
-                    <box size="0.02 0.06 0.275"/>
+                    <box size="0.02 0.06 ${tote_finger_length}"/>
                 </geometry>
-                <origin xyz="0 0 0.1375" rpy="0 0 0"/>
+                <origin xyz="0 0 ${tote_finger_length / 2}" rpy="0 0 0"/>
             </collision>
         </xacro:unless>
@@ -181,5 +167,5 @@
         <parent link="left_gripper_base_link"/>
         <child link="left_gripper_tcp"/>
-        <origin xyz="0 0 0.18" rpy="1.5708 0 0"/>
+        <origin xyz="0 0 0.14" rpy="1.5708 0 0"/>
     </joint>
 </robot>

File: src/zhishu_robot_description/urdf/zhishu_robot_description_dh.urdf (robot description, URDF)
Before this commit: robot zhishu_robot_description, 30 links, 29 joints
Links:
- link base_link: mass 11.9793854739169 -> ${11.9793854739169 * chassis_mass_scale}
- link waist_pitch_link: geometry collision box size=0.270 0.280 0.500; visual mesh filename=package://zhishu_robot_description/meshes/waist_pitch_link.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
- link waist_up_down_link: geometry collision box size=0.220 0.220 0.500; visual mesh filename=package://zhishu_robot_description/meshes/waist_up_down_lin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
Joints:
- joint right_wheel_joint: axis 0 -1 0 -> (none)
- joint waist_pitch_joint: limit lower=-0.7854 upper=0.2618 effort=100.0 velocity=1.0 -> lower=-1.57079632679 upper=0.2618 effort=${float('$(arg mobile_base_sim_waist_effort)') if '$(arg mobile_base_sim_enabled)' == 'true' else 100.0} velocity=1.0

File: src/zhishu_robot_moveit_config/config/zhishu_robot.gazebo.ros2_control.xacro (robot description, xacro)
@@ -15,4 +15,5 @@
                     <param name="initial_value">${initial_positions['left_shoulder_pitch_joint']}</param>
                 </state_interface>
+                <state_interface name="velocity"/>
             </joint>
             <joint name="left_shoulder_roll_joint">
@@ -21,4 +22,5 @@
                     <param name="initial_value">${initial_positions['left_shoulder_roll_joint']}</param>
                 </state_interface>
+                <state_interface name="velocity"/>
             </joint>
             <joint name="left_shoulder_yaw_joint">
@@ -27,4 +29,5 @@
                     <param name="initial_value">${initial_positions['left_shoulder_yaw_joint']}</param>
                 </state_interface>
+                <state_interface name="velocity"/>
             </joint>
             <joint name="left_elbow_pitch_joint">
@@ -33,4 +36,5 @@
                     <param name="initial_value">${initial_positions['left_elbow_pitch_joint']}</param>
                 </state_interface>
+                <state_interface name="velocity"/>
             </joint>
             <joint name="left_wrist_yaw_joint">
@@ -39,4 +43,5 @@
                     <param name="initial_value">${initial_positions['left_wrist_yaw_joint']}</param>
                 </state_interface>
+                <state_interface name="velocity"/>
             </joint>
             <joint name="left_wrist_pitch_joint">
@@ -45,4 +50,5 @@
                     <param name="initial_value">${initial_positions['left_wrist_pitch_joint']}</param>
                 </state_interface>
+                <state_interface name="velocity"/>
             </joint>
             <joint name="left_wrist_roll_joint">
@@ -51,4 +57,5 @@
                     <param name="initial_value">${initial_positions['left_wrist_roll_joint']}</param>
                 </state_interface>
+                <state_interface name="velocity"/>
             </joint>
             <joint name="right_shoulder_pitch_joint">
@@ -57,4 +64,5 @@
                     <param name="initial_value">${initial_positions['right_shoulder_pitch_joint']}</param>
                 </state_interface>
+                <state_interface name="velocity"/>
             </joint>
             <joint name="right_shoulder_roll_joint">
@@ -63,4 +71,5 @@
                     <param name="initial_value">${initial_positions['right_shoulder_roll_joint']}</param>
                 </state_interface>
+                <state_interface name="velocity"/>
             </joint>
             <joint name="right_shoulder_yaw_joint">
@@ -69,4 +78,5 @@
                     <param name="initial_value">${initial_positions['right_shoulder_yaw_joint']}</param>
                 </state_interface>
+                <state_interface name="velocity"/>
             </joint>
             <joint name="right_elbow_pitch_joint">
@@ -75,4 +85,5 @@
                     <param name="initial_value">${initial_positions['right_elbow_pitch_joint']}</param>
                 </state_interface>
+                <state_interface name="velocity"/>
             </joint>
             <joint name="right_wrist_yaw_joint">
@@ -81,4 +92,5 @@
                     <param name="initial_value">${initial_positions['right_wrist_yaw_joint']}</param>
                 </state_interface>
+                <state_interface name="velocity"/>
             </joint>
             <joint name="right_wrist_pitch_joint">
@@ -87,4 +99,5 @@
                     <param name="initial_value">${initial_positions['right_wrist_pitch_joint']}</param>
                 </state_interface>
+                <state_interface name="velocity"/>
             </joint>
             <joint name="right_wrist_roll_joint">
@@ -93,4 +106,5 @@
                     <param name="initial_value">${initial_positions['right_wrist_roll_joint']}</param>
                 </state_interface>
+                <state_interface name="velocity"/>
             </joint>
             <joint name="left_gripper_left_finger_joint">
@@ -105,4 +119,14 @@
                     <param name="initial_value">${initial_positions['gripper_left_finger_joint']}</param>
                 </state_interface>
+            </joint>
+            <!-- Include passive mimic fingers in Gazebo hardware info.
+                 URDF mimic alone does not register their simulated drive. -->
+            <joint name="gripper_right_finger_joint">
+                <state_interface name="position"/>
+                <state_interface name="velocity"/>
+            </joint>
+            <joint name="left_gripper_right_finger_joint">
+                <state_interface name="position"/>
+                <state_interface name="velocity"/>
             </joint>
             <joint name="waist_up_down_joint">

File: src/zhishu_robot_moveit_config/config/zhishu_robot.urdf.xacro (robot description, xacro)
@@ -81,10 +81,19 @@
             <plugin filename="libgz_ros2_control-system.so" name="gz_ros2_control::GazeboSimROS2ControlPlugin">
                 <parameters>$(find zhishu_robot_moveit_config)/config/ros2_controllers.yaml</parameters>
+                <parameters>$(find zhishu_robot_moveit_config)/config/gazebo_controller_manager.yaml</parameters>
                 <!-- Hold all joints at their configured initial positions while
                      the admittance launch loads and atomically activates controllers. -->
                 <hold_joints>true</hold_joints>
-                <position_proportional_gain>1.0</position_proportional_gain>
+                <!-- gz_ros2_control scales position error by update_rate;
+                     a sub-unit gain damps discrete contact tracking. -->
+                <position_proportional_gain>0.2</position_proportional_gain>
             </plugin>
             <xacro:if value="$(arg mobile_base_sim_enabled)">
+                <plugin filename="gz-sim-pose-publisher-system" name="gz::sim::systems::PosePublisher">
+                    <publish_model_pose>true</publish_model_pose>
+                    <publish_link_pose>false</publish_link_pose>
+                    <use_pose_vector_msg>false</use_pose_vector_msg>
+                    <update_frequency>20</update_frequency>
+                </plugin>
                 <!-- Simulation-only mobile base. The wheel joints are state-only in
                      gz_ros2_control, so DiffDrive is the sole wheel command writer. -->
@@ -102,20 +111,4 @@
                 </plugin>
             </xacro:if>
-            <!-- Extraction runs start already aligned with r0_c0.  Add
-                 wheel damping/contact friction so arm reaction forces do not
-                 roll the chassis away from the 20 cm station while the hook
-                 trajectory is executing. -->
-            <gazebo reference="left_wheel_link">
-                <mu1>8.0</mu1>
-                <mu2>8.0</mu2>
-                <kp>1000000.0</kp>
-                <kd>100.0</kd>
-            </gazebo>
-            <gazebo reference="right_wheel_link">
-                <mu1>8.0</mu1>
-                <mu2>8.0</mu2>
-                <kp>1000000.0</kp>
-                <kd>100.0</kd>
-            </gazebo>
             <xacro:if value="$(arg bottle_grasp_sim_enabled)">
                 <!-- Contact determines closure timing; this simulation-only
@@ -132,4 +125,29 @@
             </xacro:if>
         </gazebo>
+        <!-- Link-specific extensions must be robot-level siblings, not nested
+             in the model-level plugin gazebo tag: sdformat otherwise ignores
+             these friction values and copies them as unsupported children. -->
+        <xacro:if value="$(arg mobile_base_sim_enabled)">
+            <gazebo reference="left_wheel_link"><mu1>8.0</mu1><mu2>8.0</mu2><kp>1000000.0</kp><kd>100.0</kd></gazebo>
+            <gazebo reference="right_wheel_link"><mu1>8.0</mu1><mu2>8.0</mu2><kp>1000000.0</kp><kd>100.0</kd></gazebo>
+            <!-- Candidate rubber pads: still require physical calibration. -->
+            <gazebo reference="gripper_left_finger_link"><mu1>3.0</mu1><mu2>3.0</mu2></gazebo>
+            <gazebo reference="gripper_right_finger_link"><mu1>3.0</mu1><mu2>3.0</mu2></gazebo>
+            <gazebo reference="left_gripper_left_finger_link"><mu1>3.0</mu1><mu2>3.0</mu2></gazebo>
+            <gazebo reference="left_gripper_right_finger_link"><mu1>3.0</mu1><mu2>3.0</mu2></gazebo>
+            <xacro:macro name="pallet_contact_sensor" params="link">
+                <gazebo reference="${link}">
+                    <sensor name="${link}_contact" type="contact">
+                        <always_on>true</always_on><update_rate>50</update_rate>
+                        <topic>/pallet_contacts/${link}</topic>
+                        <contact><collision>${link}_collision</collision></contact>
+                    </sensor>
+                </gazebo>
+            </xacro:macro>
+            <xacro:pallet_contact_sensor link="right_shoulder_pitch_link"/>
+            <xacro:pallet_contact_sensor link="right_elbow_pitch_link"/>
+            <xacro:pallet_contact_sensor link="gripper_left_finger_link"/>
+            <xacro:pallet_contact_sensor link="gripper_right_finger_link"/>
+        </xacro:if>
     </xacro:if>
 </robot>

Commit message: feat(grasp): 增加15kg料箱落底松爪与低速转运（360mm夹爪，TCP300mm，弯腰下限-45°，实际最大约-44.98°）

File: src/zhishu_robot_description/urdf/gripper.xacro (robot description, xacro)
@@ -1,5 +1,6 @@
 <?xml version='1.0' encoding='UTF-8'?>
 <robot xmlns:xacro="http://www.ros.org/wiki/xacro">
-    <xacro:property name="tote_finger_length" value="0.200"/>
+    <xacro:arg name="tote_finger_length" default="0.200"/>
+    <xacro:property name="tote_finger_length" value="${float('$(arg tote_finger_length)')}"/>
     <!-- Gazebo Sim only creates dynamic links that have valid inertial data.
          Without this block the finger links, their prismatic joints, and the
@@ -7,5 +8,5 @@
     <xacro:macro name="gripper_finger_inertial">
         <inertial>
-            <!-- Candidate 200 mm fingers; TCP is 80 mm behind the tip.
+            <!-- Configurable fingers; TCP is 80 mm behind the tip.
                  The tote grasp target limits insertion to about 50 mm. -->
             <origin xyz="0 0 ${tote_finger_length / 2}" rpy="0 0 0"/>
@@ -89,5 +90,5 @@
         <parent link="gripper_base_link"/>
         <child link="right_gripper_tcp"/>
-        <origin xyz="0 0 0.14" rpy="1.5708 0 0"/>
+        <origin xyz="0 0 ${tote_finger_length - 0.060}" rpy="1.5708 0 0"/>
     </joint>
     <!-- Left gripper: same geometry and kinematics as the right gripper, but with left_* names. -->
@@ -167,5 +168,5 @@
         <parent link="left_gripper_base_link"/>
         <child link="left_gripper_tcp"/>
-        <origin xyz="0 0 0.14" rpy="1.5708 0 0"/>
+        <origin xyz="0 0 ${tote_finger_length - 0.060}" rpy="1.5708 0 0"/>
     </joint>
 </robot>

File: src/zhishu_robot_description/urdf/zhishu_robot_description_dh.urdf (robot description, URDF)
Before this commit: robot zhishu_robot_description, 30 links, 29 joints
Joints:
- joint waist_pitch_joint: limit lower=-1.57079632679 upper=0.2618 effort=${float('$(arg mobile_base_sim_waist_effort)') if '$(arg mobile_base_sim_enabled)' == 'true' else 100.0} velocity=1.0 -> lower=$(arg waist_pitch_min) upper=0.2618 effort=${float('$(arg mobile_base_sim_waist_effort)') if '$(arg mobile_base_sim_enabled)' == 'true' else 100.0} velocity=1.0

Commit message: feat(grasp): 完成对面推箱与双臂转运
360mm手指，推送TCP380mm、抓取TCP300mm；弯腰下限-90°，实测最低约-89.99°。修复控制插件空状态崩溃、起身轨迹与双爪开度复位，完整验证及录像重跑通过。

File: src/zhishu_robot_description/urdf/gripper.xacro (robot description, xacro)
@@ -87,4 +87,10 @@
     </joint>
     <link name="right_gripper_tcp"/>
+    <link name="right_gripper_push_tip"/>
+    <joint name="right_gripper_push_tip_joint" type="fixed">
+        <parent link="gripper_base_link"/>
+        <child link="right_gripper_push_tip"/>
+        <origin xyz="0 0 ${tote_finger_length + 0.020}" rpy="1.5708 0 0"/>
+    </joint>
     <joint name="right_gripper_tcp_joint" type="fixed">
         <parent link="gripper_base_link"/>
