Commit message: 初步调通右臂七个电机

File: src/zhishu_robot_description/urdf/zhishu_robot_description_dh.urdf (robot description, URDF)
Before this commit: robot zhishu_robot_description, 30 links, 29 joints
Links:
- link waist_pitch_link: geometry collision box size=0.30 0.33 0.560; visual mesh filename=package://zhishu_robot_description/meshes/waist_pitch_link.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
Joints:
- joint right_shoulder_roll_joint: axis 0 0 1 -> 0 0 -1
- joint right_shoulder_yaw_joint: axis 0 0 1 -> 0 0 -1
- joint right_wrist_pitch_joint: axis 0 0 1 -> 0 0 -1

File: src/zhishu_robot_moveit_config/config/zhishu_robot.ros2_control.xacro (robot description, xacro)
@@ -9,7 +9,35 @@
                 <!-- <param name="calculate_dynamics">true</param> -->
                 <plugin>es_motor_hardware/EsMotorHardwareInterface</plugin>
+                <!-- IgH EtherCAT / GH1 SERVOPACK defaults. Per-joint params below can override these. -->
+                <param name="cycle_ns">1000000</param>
+                <param name="enable_dc">true</param>
+                <param name="assign_activate">0x0300</param>
+                <param name="sync0_shift_ns">622620</param>
+                <param name="select_dc_reference_clock">true</param>
+                <param name="dc_reference_alias">0</param>
+                <param name="dc_reference_slave_position">0</param>
+                <param name="enable_realtime">true</param>
+                <param name="realtime_priority">80</param>
+                <param name="master_index">0</param>
+                <param name="alias">0</param>
+                <param name="vendor_id">0x00206688</param>
+                <param name="product_code">0x26483052</param>
+                <param name="configure_sdo">true</param>
+                <param name="configure_pdos">true</param>
+                <param name="mode_of_operation">8</param>
+                <param name="auto_enable">false</param>
+                <param name="auto_fault_reset">true</param>
+                <param name="counts_per_rev">131072.0</param>
+                <param name="max_velocity_counts_s">8000.0</param>
+                <param name="max_accel_counts_s2">20000.0</param>
+                <param name="target_tolerance_counts">20</param>
+                <param name="joint_sign">1.0</param>
+                <param name="position_offset_rad">0.0</param>
             </hardware>
             <!-- right_arm -->
             <joint name="right_shoulder_pitch_joint">
+                <param name="use_ethercat">true</param>
+                <param name="motor_name">right_arm_motor_0</param>
+                <param name="slave_position">0</param>
                 <command_interface name="position"/>
                 <state_interface name="position">
@@ -18,4 +46,7 @@
             </joint>
             <joint name="right_shoulder_roll_joint">
+                <param name="use_ethercat">true</param>
+                <param name="motor_name">right_arm_motor_1</param>
+                <param name="slave_position">1</param>
                 <command_interface name="position"/>
                 <state_interface name="position">
@@ -24,4 +55,7 @@
             </joint>
             <joint name="right_shoulder_yaw_joint">
+                <param name="use_ethercat">true</param>
+                <param name="motor_name">right_arm_motor_2</param>
+                <param name="slave_position">2</param>
                 <command_interface name="position"/>
                 <state_interface name="position">
@@ -30,4 +64,7 @@
             </joint>
             <joint name="right_elbow_pitch_joint">
+                <param name="use_ethercat">true</param>
+                <param name="motor_name">right_arm_motor_3</param>
+                <param name="slave_position">3</param>
                 <command_interface name="position"/>
                 <state_interface name="position">
@@ -36,4 +73,7 @@
             </joint>
             <joint name="right_wrist_yaw_joint">
+                <param name="use_ethercat">true</param>
+                <param name="motor_name">right_arm_motor_4</param>
+                <param name="slave_position">4</param>
                 <command_interface name="position"/>
                 <state_interface name="position">
@@ -42,4 +82,7 @@
             </joint>
             <joint name="right_wrist_pitch_joint">
+                <param name="use_ethercat">true</param>
+                <param name="motor_name">right_arm_motor_5</param>
+                <param name="slave_position">5</param>
                 <command_interface name="position"/>
                 <state_interface name="position">
@@ -48,4 +91,7 @@
             </joint>
             <joint name="right_wrist_roll_joint">
+                <param name="use_ethercat">true</param>
+                <param name="motor_name">right_arm_motor_6</param>
+                <param name="slave_position">6</param>
                 <command_interface name="position"/>
                 <state_interface name="position">

File: src/zhishu_robot_moveit_config/config/zhishu_robot.urdf.xacro (robot description, xacro)
@@ -6,4 +6,4 @@
     <!-- Import control_xacro -->
     <xacro:include filename="zhishu_robot.ros2_control.xacro" />
-    <xacro:zhishu_robot_ros2_control name="FakeSystem" initial_positions_file="$(arg initial_positions_file)"/>
+    <xacro:zhishu_robot_ros2_control name="RightArmEtherCATSystem" initial_positions_file="$(arg initial_positions_file)"/>
 </robot>

Commit message: 硬件联调左机械臂

File: src/zhishu_robot_description/urdf/zhishu_robot_description_dh.urdf (robot description, URDF)
Before this commit: robot zhishu_robot_description, 30 links, 29 joints
Joints:
- joint left_shoulder_roll_joint: axis 0 0 1 -> 0 0 -1
- joint left_shoulder_yaw_joint: axis 0 0 1 -> 0 0 -1
- joint left_wrist_pitch_joint: axis 0 0 1 -> 0 0 -1

File: src/zhishu_robot_moveit_config/config/zhishu_robot.right_arm.ros2_control.xacro (robot description, xacro)
@@ -1,12 +1,12 @@
 <?xml version="1.0"?>
 <robot xmlns:xacro="http://www.ros.org/wiki/xacro">
-    <xacro:macro name="zhishu_robot_ros2_control" params="name initial_positions_file">
+    <xacro:macro name="zhishu_robot_right_arm_ros2_control" params="name initial_positions_file">
         <xacro:property name="initial_positions" value="${load_yaml(initial_positions_file)['initial_positions']}"/>
         <ros2_control name="${name}" type="system">
             <hardware>
                 <!-- By default, set up controllers for simulation. This won't work on real hardware -->
-                <!-- <plugin>mock_components/GenericSystem</plugin> -->
-                <!-- <param name="calculate_dynamics">true</param> -->
-                <plugin>es_motor_hardware/EsMotorHardwareInterface</plugin>
+                <plugin>mock_components/GenericSystem</plugin>
+                <param name="calculate_dynamics">true</param>
+                <!-- <plugin>es_motor_hardware/EsMotorHardwareInterface</plugin> -->
                 <!-- IgH EtherCAT / GH1 SERVOPACK defaults. Per-joint params below can override these. -->
                 <param name="cycle_ns">4000000</param>
@@ -99,48 +99,5 @@
                 </state_interface>
             </joint>
-            <!-- left_arm -->
-            <joint name="left_shoulder_pitch_joint">
-                <command_interface name="position"/>
-                <state_interface name="position">
-                  <param name="initial_value">${initial_positions['left_shoulder_pitch_joint']}</param>
-                </state_interface>
-            </joint>
-            <joint name="left_shoulder_roll_joint">
-                <command_interface name="position"/>
-                <state_interface name="position">
-                  <param name="initial_value">${initial_positions['left_shoulder_roll_joint']}</param>
-                </state_interface>
-            </joint>
-            <joint name="left_shoulder_yaw_joint">
-                <command_interface name="position"/>
-                <state_interface name="position">
-                  <param name="initial_value">${initial_positions['left_shoulder_yaw_joint']}</param>
-                </state_interface>
-            </joint>
-            <joint name="left_elbow_pitch_joint">
-                <command_interface name="position"/>
-                <state_interface name="position">
-                  <param name="initial_value">${initial_positions['left_elbow_pitch_joint']}</param>
-                </state_interface>
-            </joint>
-            <joint name="left_wrist_yaw_joint">
-                <command_interface name="position"/>
-                <state_interface name="position">
-                  <param name="initial_value">${initial_positions['left_wrist_yaw_joint']}</param>
-                </state_interface>
-            </joint>
-            <joint name="left_wrist_pitch_joint">
-                <command_interface name="position"/>
-                <state_interface name="position">
-                  <param name="initial_value">${initial_positions['left_wrist_pitch_joint']}</param>
-                </state_interface>
-            </joint>
-            <joint name="left_wrist_roll_joint">
-                <command_interface name="position"/>
-                <state_interface name="position">
-                  <param name="initial_value">${initial_positions['left_wrist_roll_joint']}</param>
-                </state_interface>
-            </joint>
-            <joint name="gripper_left_finger_joint">
+            <!-- <joint name="gripper_left_finger_joint">
                 <command_interface name="position"/>
                 <state_interface name="position">
@@ -177,5 +134,5 @@
                   <param name="initial_value">${initial_positions['right_wheel_joint']}</param>
                 </state_interface>
-            </joint>
+            </joint> -->
         </ros2_control>
     </xacro:macro>

File: src/zhishu_robot_moveit_config/config/zhishu_robot.urdf.xacro (robot description, xacro)
@@ -5,5 +5,7 @@
     <xacro:include filename="$(find zhishu_robot_description)/urdf/zhishu_robot.urdf.xacro" />
     <!-- Import control_xacro -->
-    <xacro:include filename="zhishu_robot.ros2_control.xacro" />
-    <xacro:zhishu_robot_ros2_control name="RightArmEtherCATSystem" initial_positions_file="$(arg initial_positions_file)"/>
+    <xacro:include filename="zhishu_robot.left_arm.ros2_control.xacro" />
+    <xacro:include filename="zhishu_robot.right_arm.ros2_control.xacro" />
+    <xacro:zhishu_robot_left_arm_ros2_control name="LeftArmEtherCATSystem" initial_positions_file="$(arg initial_positions_file)"/>
+    <xacro:zhishu_robot_right_arm_ros2_control name="RightArmEtherCATSystem" initial_positions_file="$(arg initial_positions_file)"/>
 </robot>
