Commit message: 双臂mtc修正部分参数

File: src/zhishu_robot_description/urdf/zhishu_robot_description_dh.urdf (robot description, URDF)
Before this commit: robot zhishu_robot_description, 30 links, 29 joints
Links:
- link waist_pitch_link: geometry collision box size=0.30 0.31 0.560; visual mesh filename=package://zhishu_robot_description/meshes/waist_pitch_link.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

File: src/zhishu_robot_moveit_config/config/zhishu_robot.left_arm.ros2_control.xacro (robot description, xacro)
@@ -6,7 +6,7 @@
             <hardware>
                 <!-- By default, set up controllers for simulation. This won't work on real hardware -->
-                <plugin>mock_components/GenericSystem</plugin>
-                <param name="calculate_dynamics">true</param>
-                <!-- <plugin>left_es_motor_hardware/LeftEsMotorHardwareInterface</plugin> -->
+                <!-- <plugin>mock_components/GenericSystem</plugin> -->
+                <!-- <param name="calculate_dynamics">true</param> -->
+                <plugin>left_es_motor_hardware/LeftEsMotorHardwareInterface</plugin>
                 <!-- IgH EtherCAT / GH1 SERVOPACK defaults. Per-joint params below can override these. -->
                 <param name="cycle_ns">2000000</param>

File: src/zhishu_robot_moveit_config/config/zhishu_robot.right_arm.ros2_control.xacro (robot description, xacro)
@@ -6,7 +6,7 @@
             <hardware>
                 <!-- By default, set up controllers for simulation. This won't work on real hardware -->
-                <plugin>mock_components/GenericSystem</plugin>
-                <param name="calculate_dynamics">true</param>
-                <!-- <plugin>es_motor_hardware/EsMotorHardwareInterface</plugin> -->
+                <!-- <plugin>mock_components/GenericSystem</plugin> -->
+                <!-- <param name="calculate_dynamics">true</param> -->
+                <plugin>es_motor_hardware/EsMotorHardwareInterface</plugin>
                 <!-- IgH EtherCAT / GH1 SERVOPACK defaults. Per-joint params below can override these. -->
                 <param name="cycle_ns">2000000</param>

Commit message: 修正双臂2轴的上下限

File: src/zhishu_robot_description/urdf/zhishu_robot_description_dh.urdf (robot description, URDF)
Before this commit: robot zhishu_robot_description, 30 links, 29 joints
Joints:
- joint left_shoulder_roll_joint: limit lower=-0.43633 upper=1.4835 effort=100.0 velocity=1.0 -> lower=-1.4835 upper=0.43633 effort=100.0 velocity=1.0
- joint right_shoulder_roll_joint: limit lower=-1.4835 upper=0.43633 effort=100.0 velocity=1.0 -> lower=-0.43633 upper=1.4835 effort=100.0 velocity=1.0
