Commit message: fanshou dual mtc

File: src/zhishu_robot_description/urdf/zhishu_robot.gazebo.urdf.xacro (robot description, xacro)
@@ -7,10 +7,10 @@
         <parent link="L_hand_link" />
         <child link="left_gripper_base_link" />
-        <origin xyz="0 0 0" rpy="0 3.14159 0" />
+        <origin xyz="0 0 0" rpy="0 3.14159 1.570796327" />
     </joint>
     <joint name="right_gripper_joint" type="fixed">
         <parent link="R_hand_link" />
         <child link="gripper_base_link" />
-        <origin xyz="0 0 0" rpy="0 3.14159 0" />
+        <origin xyz="0 0 0" rpy="0 3.14159 -1.570796327" />
     </joint>
     <xacro:include filename="$(find zhishu_robot_description)/urdf/gazebo_sim_ros2_control.urdf.xacro" />

File: src/zhishu_robot_description/urdf/zhishu_robot.urdf.xacro (robot description, xacro)
@@ -7,10 +7,10 @@
         <parent link="L_hand_link" />
         <child link="left_gripper_base_link" />
-        <origin xyz="0 0 0" rpy="0 3.14159 0" />
+        <origin xyz="0 0 0" rpy="0 3.14159 1.570796327" />
     </joint>
     <joint name="right_gripper_joint" type="fixed">
         <parent link="R_hand_link" />
         <child link="gripper_base_link" />
-        <origin xyz="0 0 0" rpy="0 3.14159 0" />
+        <origin xyz="0 0 0" rpy="0 3.14159 -1.570796327" />
     </joint>
 </robot>

File: src/zhishu_robot_moveit_config/config/zhishu_robot.right_arm.ros2_control.xacro (robot description, xacro)
@@ -6,7 +6,7 @@
             <hardware>
                 <!-- By default, set up controllers for simulation. This won't work on real hardware -->
-                <plugin>mock_components/GenericSystem</plugin>
-                <param name="calculate_dynamics">true</param>
-                <!-- <plugin>es_motor_hardware/EsMotorHardwareInterface</plugin> -->
+                <!-- <plugin>mock_components/GenericSystem</plugin> -->
+                <!-- <param name="calculate_dynamics">true</param> -->
+                <plugin>es_motor_hardware/EsMotorHardwareInterface</plugin>
                 <!-- IgH EtherCAT / GH1 SERVOPACK defaults. Per-joint params below can override these. -->
                 <param name="cycle_ns">2000000</param>
