Commit message: 由humble升级到jazzy

File: src/zhishu_robot_description/urdf/gazebo_sim_ros2_control.urdf.xacro (robot description, xacro)
@@ -4,6 +4,6 @@
         <xacro:if value="${use_gazebo}">
             <gazebo>
-                <plugin filename="gz_ros2_control-system" name="gz_ros2_control::GazeboSimROS2ControlPlugin">
-                    <parameters>$(find zhishu_moveit_config)/config/ros2_controllers.yaml</parameters>
+                <plugin filename="libgz_ros2_control-system.so" name="gz_ros2_control::GazeboSimROS2ControlPlugin">
+                    <parameters>$(find zhishu_robot_moveit_config)/config/ros2_controllers.yaml</parameters>
                     <ros>
                         <remapping>/controller_manager/robot_description:=/robot_description</remapping>

File: src/zhishu_robot_description/urdf/gripper.xacro (robot description, xacro)
@@ -1,4 +1,17 @@
 <?xml version='1.0' encoding='UTF-8'?>
 <robot xmlns:xacro="http://www.ros.org/wiki/xacro">
+    <!-- Gazebo Sim only creates dynamic links that have valid inertial data.
+         Without this block the finger links, their prismatic joints, and the
+         corresponding ros2_control command interfaces are omitted from SDF. -->
+    <xacro:macro name="gripper_finger_inertial">
+        <inertial>
+            <origin xyz="0 0 0.10" rpy="0 0 0"/>
+            <mass value="0.1"/>
+            <inertia
+                ixx="0.000363333" ixy="0.0" ixz="0.0"
+                iyy="0.000336667" iyz="0.0"
+                izz="0.000033333"/>
+        </inertial>
+    </xacro:macro>
     <link name="gripper_base_link">
         <visual>
@@ -17,4 +30,5 @@
     </link>
     <link name="gripper_left_finger_link">
+        <xacro:gripper_finger_inertial/>
         <visual>
             <geometry>
@@ -32,4 +46,5 @@
     </link>
     <link name="gripper_right_finger_link">
+        <xacro:gripper_finger_inertial/>
         <visual>
             <geometry>
@@ -84,4 +99,5 @@
     </link>
     <link name="left_gripper_left_finger_link">
+        <xacro:gripper_finger_inertial/>
         <visual>
             <geometry>
@@ -99,4 +115,5 @@
     </link>
     <link name="left_gripper_right_finger_link">
+        <xacro:gripper_finger_inertial/>
         <visual>
             <geometry>

File: src/zhishu_robot_moveit_config/config/zhishu_robot.left_arm.ros2_control.xacro (robot description, xacro)
@@ -1,12 +1,20 @@
 <?xml version="1.0"?>
 <robot xmlns:xacro="http://www.ros.org/wiki/xacro">
-    <xacro:macro name="zhishu_robot_left_arm_ros2_control" params="name initial_positions_file">
-        <xacro:property name="initial_positions" value="${load_yaml(initial_positions_file)['initial_positions']}"/>
+    <xacro:macro name="zhishu_robot_left_arm_ros2_control" params="name initial_positions_file use_gazebo:=false use_fake_hardware:=true">
+        <xacro:property name="initial_positions" value="${xacro.load_yaml(initial_positions_file)['initial_positions']}"/>
         <ros2_control name="${name}" type="system">
             <hardware>
-                <!-- By default, set up controllers for simulation. This won't work on real hardware -->
-                <plugin>mock_components/GenericSystem</plugin>
-                <param name="calculate_dynamics">true</param>
-                <!-- <plugin>left_es_motor_hardware/LeftEsMotorHardwareInterface</plugin> -->
+                <xacro:if value="${use_gazebo}">
+                    <plugin>gz_ros2_control/GazeboSimSystem</plugin>
+                </xacro:if>
+                <xacro:unless value="${use_gazebo}">
+                    <xacro:if value="${use_fake_hardware}">
+                        <plugin>mock_components/GenericSystem</plugin>
+                        <param name="calculate_dynamics">true</param>
+                    </xacro:if>
+                    <xacro:unless value="${use_fake_hardware}">
+                        <plugin>left_es_motor_hardware/LeftEsMotorHardwareInterface</plugin>
+                    </xacro:unless>
+                </xacro:unless>
                 <!-- IgH EtherCAT / GH1 SERVOPACK defaults. Per-joint params below can override these. -->
                 <param name="cycle_ns">2000000</param>
@@ -110,6 +118,6 @@
                 </state_interface>
             </joint>
-            <!-- Keep both non-EtherCAT gripper command interfaces in one mock
-                 hardware component. GenericSystem on ROS 2 Humble receives the
+            <!-- Keep both non-EtherCAT gripper command interfaces in one
+                 hardware component. GenericSystem receives the
                  complete mode-switch request and rejects foreign gripper joints
                  when the two grippers are split across different components. -->

File: src/zhishu_robot_moveit_config/config/zhishu_robot.right_arm.ros2_control.xacro (robot description, xacro)
@@ -1,12 +1,20 @@
 <?xml version="1.0"?>
 <robot xmlns:xacro="http://www.ros.org/wiki/xacro">
-    <xacro:macro name="zhishu_robot_right_arm_ros2_control" params="name initial_positions_file">
-        <xacro:property name="initial_positions" value="${load_yaml(initial_positions_file)['initial_positions']}"/>
+    <xacro:macro name="zhishu_robot_right_arm_ros2_control" params="name initial_positions_file use_gazebo:=false use_fake_hardware:=true">
+        <xacro:property name="initial_positions" value="${xacro.load_yaml(initial_positions_file)['initial_positions']}"/>
         <ros2_control name="${name}" type="system">
             <hardware>
-                <!-- By default, set up controllers for simulation. This won't work on real hardware -->
-                <plugin>mock_components/GenericSystem</plugin>
-                <param name="calculate_dynamics">true</param>
-                <!-- <plugin>es_motor_hardware/EsMotorHardwareInterface</plugin> -->
+                <xacro:if value="${use_gazebo}">
+                    <plugin>gz_ros2_control/GazeboSimSystem</plugin>
+                </xacro:if>
+                <xacro:unless value="${use_gazebo}">
+                    <xacro:if value="${use_fake_hardware}">
+                        <plugin>mock_components/GenericSystem</plugin>
+                        <param name="calculate_dynamics">true</param>
+                    </xacro:if>
+                    <xacro:unless value="${use_fake_hardware}">
+                        <plugin>es_motor_hardware/EsMotorHardwareInterface</plugin>
+                    </xacro:unless>
+                </xacro:unless>
                 <!-- IgH EtherCAT / GH1 SERVOPACK defaults. Per-joint params below can override these. -->
                 <param name="cycle_ns">2000000</param>

File: src/zhishu_robot_moveit_config/config/zhishu_robot.urdf.xacro (robot description, xacro)
@@ -2,4 +2,6 @@
 <robot xmlns:xacro="http://www.ros.org/wiki/xacro" name="zhishu_robot">
     <xacro:arg name="initial_positions_file" default="initial_positions.yaml" />
+    <xacro:arg name="use_gazebo" default="false" />
+    <xacro:arg name="use_fake_hardware" default="true" />
     <!-- Import zhishu_robot urdf file -->
     <xacro:include filename="$(find zhishu_robot_description)/urdf/zhishu_robot.urdf.xacro" />
@@ -7,5 +9,24 @@
     <xacro:include filename="zhishu_robot.left_arm.ros2_control.xacro" />
     <xacro:include filename="zhishu_robot.right_arm.ros2_control.xacro" />
-    <xacro:zhishu_robot_left_arm_ros2_control name="LeftArmEtherCATSystem" initial_positions_file="$(arg initial_positions_file)"/>
-    <xacro:zhishu_robot_right_arm_ros2_control name="RightArmEtherCATSystem" initial_positions_file="$(arg initial_positions_file)"/>
+    <xacro:include filename="zhishu_robot.gazebo.ros2_control.xacro" />
+    <xacro:unless value="$(arg use_gazebo)">
+        <xacro:zhishu_robot_left_arm_ros2_control
+            name="LeftArmSystem"
+            initial_positions_file="$(arg initial_positions_file)"
+            use_fake_hardware="$(arg use_fake_hardware)"/>
+        <xacro:zhishu_robot_right_arm_ros2_control
+            name="RightArmSystem"
+            initial_positions_file="$(arg initial_positions_file)"
+            use_fake_hardware="$(arg use_fake_hardware)"/>
+    </xacro:unless>
+    <xacro:if value="$(arg use_gazebo)">
+        <xacro:zhishu_robot_gazebo_ros2_control
+            name="GazeboSystem"
+            initial_positions_file="$(arg initial_positions_file)"/>
+        <gazebo>
+            <plugin filename="libgz_ros2_control-system.so" name="gz_ros2_control::GazeboSimROS2ControlPlugin">
+                <parameters>$(find zhishu_robot_moveit_config)/config/ros2_controllers.yaml</parameters>
+            </plugin>
+        </gazebo>
+    </xacro:if>
 </robot>
