Commit message: feat(admittance): 新增双臂导纳控制并增加Gazebo搬箱场景

File: src/zhishu_robot_description/urdf/zhishu_robot.urdf.xacro (robot description, xacro)
@@ -4,4 +4,30 @@
     <xacro:include filename="$(find zhishu_robot_description)/urdf/gripper.xacro"/>
     <xacro:include filename="$(find zhishu_robot_description)/urdf/zhishu_robot_description_dh.urdf"/>
+    <!-- Preserve the wrist-to-hand fixed joints in Gazebo so their reaction
+         wrench can be measured by simulated six-axis force/torque sensors. -->
+    <gazebo reference="L_hand_joint">
+        <preserveFixedJoint>true</preserveFixedJoint>
+        <sensor name="left_wrist_ft" type="force_torque">
+            <always_on>true</always_on>
+            <update_rate>250</update_rate>
+            <topic>/left_wrist_ft</topic>
+            <force_torque>
+                <frame>child</frame>
+                <measure_direction>child_to_parent</measure_direction>
+            </force_torque>
+        </sensor>
+    </gazebo>
+    <gazebo reference="R_hand_joint">
+        <preserveFixedJoint>true</preserveFixedJoint>
+        <sensor name="right_wrist_ft" type="force_torque">
+            <always_on>true</always_on>
+            <update_rate>250</update_rate>
+            <topic>/right_wrist_ft</topic>
+            <force_torque>
+                <frame>child</frame>
+                <measure_direction>child_to_parent</measure_direction>
+            </force_torque>
+        </sensor>
+    </gazebo>
     <joint name="left_gripper_joint" type="fixed">
         <parent link="L_hand_link" />

File: src/zhishu_robot_description/urdf/zhishu_robot_description_dh.urdf (robot description, URDF)
Before this commit: robot zhishu_robot_description, 30 links, 29 joints
Links:
- link L_hand_link: mass None -> 0.08
- link R_hand_link: mass None -> 0.08

File: src/zhishu_robot_moveit_config/config/zhishu_robot.urdf.xacro (robot description, xacro)
@@ -30,4 +30,8 @@
             <plugin filename="libgz_ros2_control-system.so" name="gz_ros2_control::GazeboSimROS2ControlPlugin">
                 <parameters>$(find zhishu_robot_moveit_config)/config/ros2_controllers.yaml</parameters>
+                <!-- Hold all joints at their configured initial positions while
+                     the admittance launch loads and atomically activates controllers. -->
+                <hold_joints>true</hold_joints>
+                <position_proportional_gain>1.0</position_proportional_gain>
             </plugin>
         </gazebo>

Commit message: feat(description): 添加手眼标定相机与标定板模型

File: src/zhishu_robot_description/urdf/zhishu_robot.urdf.xacro (robot description, xacro)
@@ -1,7 +1,12 @@
 <?xml version="1.0"?>
 <robot name="zhishu_robot" xmlns:xacro="http://www.ros.org/wiki/xacro">
+    <xacro:arg name="use_head_camera" default="false"/>
+    <xacro:arg name="hide_head_pitch_visual" default="false"/>
+    <xacro:arg name="handeye_target_enabled" default="false"/>
     <xacro:include filename="$(find zhishu_robot_description)/urdf/common_properties.xacro"/>
     <xacro:include filename="$(find zhishu_robot_description)/urdf/gripper.xacro"/>
     <xacro:include filename="$(find zhishu_robot_description)/urdf/zhishu_robot_description_dh.urdf"/>
+    <xacro:include filename="$(find zhishu_robot_description)/urdf/head_camera_handeye.xacro"/>
+    <xacro:head_camera_sensor enabled="$(arg use_head_camera)"/>
     <!-- Preserve the wrist-to-hand fixed joints in Gazebo so their reaction
          wrench can be measured by simulated six-axis force/torque sensors. -->
@@ -40,3 +45,4 @@
         <origin xyz="0 0 0" rpy="0 3.14159 -1.570796327" />
     </joint>
+    <xacro:left_handeye_target enabled="$(arg handeye_target_enabled)"/>
 </robot>

File: src/zhishu_robot_description/urdf/zhishu_robot_description_dh.urdf (robot description, URDF)
Before this commit: robot zhishu_robot_description, 30 links, 29 joints
Links:
- link head_pitch_link: geometry collision box size=0.190 0.160 0.230

File: src/zhishu_robot_moveit_config/config/zhishu_robot.urdf.xacro (robot description, xacro)
@@ -5,4 +5,7 @@
     <xacro:arg name="use_fake_hardware" default="true" />
     <xacro:arg name="enable_motors_on_activate" default="true" />
+    <xacro:arg name="use_head_camera" default="false" />
+    <xacro:arg name="hide_head_pitch_visual" default="false" />
+    <xacro:arg name="handeye_target_enabled" default="false" />
     <!-- Import zhishu_robot urdf file -->
     <xacro:include filename="$(find zhishu_robot_description)/urdf/zhishu_robot.urdf.xacro" />
