Commit message: feat(handeye): 替换 ChArUco 标定板并完善仿真退出流程
将仿真标定板更新为 7×5、DICT_4X4_50、30 mm 方格和 22 mm Marker，完善自动检测与求解，并修复 Gazebo 和 MoveGroup 退出时的崩溃及强制终止提示。

File: src/zhishu_robot_description/urdf/handeye_target_pattern.xacro (robot description, xacro)
@@ -1,894 +1,1045 @@
 <?xml version="1.0"?>
 <robot xmlns:xacro="http://www.ros.org/wiki/xacro">
-  <!-- Generated geometric 3x4 DICT_5X5_250 board. The cells are mirrored
-       on local -X because the camera observes the physical board back face. -->
+  <!-- Generated 7x5 DICT_4X4_50 ChArUco board:
+       square_length=0.030 m, marker_length=0.022 m.
+       The pattern is mirrored onto local -X because that is the camera-facing side. -->
   <xacro:macro name="handeye_target_pattern">
     <visual name="handeye_board_backing">
-      <geometry><box size="0.003 0.240 0.315"/></geometry>
+      <geometry><box size="0.003 0.2300000 0.1700000"/></geometry>
       <material name="handeye_white"><color rgba="1 1 1 1"/></material>
     </visual>
     <visual name="handeye_black_0">
-      <origin xyz="-0.00175 0.0750000 0.1382143" rpy="0 0 0"/>
-      <geometry><box size="0.0005 0.0600000 0.0085714"/></geometry>
+      <origin xyz="-0.00175 0.0900000 0.0600000" rpy="0 0 0"/>
+      <geometry><box size="0.0005 0.0300000 0.0300000"/></geometry>
       <material name="handeye_black"><color rgba="0 0 0 1"/></material>
     </visual>
     <visual name="handeye_black_1">
-      <origin xyz="-0.00175 0.1007143 0.1296429" rpy="0 0 0"/>
-      <geometry><box size="0.0005 0.0085714 0.0085714"/></geometry>
+      <origin xyz="-0.00175 0.0600000 0.0691667" rpy="0 0 0"/>
+      <geometry><box size="0.0005 0.0220000 0.0036667"/></geometry>
       <material name="handeye_black"><color rgba="0 0 0 1"/></material>
     </visual>
     <visual name="handeye_black_2">
-      <origin xyz="-0.00175 0.0835714 0.1296429" rpy="0 0 0"/>
-      <geometry><box size="0.0005 0.0085714 0.0085714"/></geometry>
+      <origin xyz="-0.00175 0.0691667 0.0655000" rpy="0 0 0"/>
+      <geometry><box size="0.0005 0.0036667 0.0036667"/></geometry>
       <material name="handeye_black"><color rgba="0 0 0 1"/></material>
     </visual>
     <visual name="handeye_black_3">
-      <origin xyz="-0.00175 0.0578571 0.1296429" rpy="0 0 0"/>
-      <geometry><box size="0.0005 0.0257143 0.0085714"/></geometry>
+      <origin xyz="-0.00175 0.0618333 0.0655000" rpy="0 0 0"/>
+      <geometry><box size="0.0005 0.0036667 0.0036667"/></geometry>
       <material name="handeye_black"><color rgba="0 0 0 1"/></material>
     </visual>
     <visual name="handeye_black_4">
-      <origin xyz="-0.00175 0.0964286 0.1210714" rpy="0 0 0"/>
-      <geometry><box size="0.0005 0.0171429 0.0085714"/></geometry>
+      <origin xyz="-0.00175 0.0508333 0.0655000" rpy="0 0 0"/>
+      <geometry><box size="0.0005 0.0036667 0.0036667"/></geometry>
       <material name="handeye_black"><color rgba="0 0 0 1"/></material>
     </visual>
     <visual name="handeye_black_5">
-      <origin xyz="-0.00175 0.0750000 0.1210714" rpy="0 0 0"/>
-      <geometry><box size="0.0005 0.0085714 0.0085714"/></geometry>
+      <origin xyz="-0.00175 0.0673333 0.0618333" rpy="0 0 0"/>
+      <geometry><box size="0.0005 0.0073333 0.0036667"/></geometry>
       <material name="handeye_black"><color rgba="0 0 0 1"/></material>
     </visual>
     <visual name="handeye_black_6">
-      <origin xyz="-0.00175 0.0492857 0.1210714" rpy="0 0 0"/>
-      <geometry><box size="0.0005 0.0085714 0.0085714"/></geometry>
+      <origin xyz="-0.00175 0.0581667 0.0618333" rpy="0 0 0"/>
+      <geometry><box size="0.0005 0.0036667 0.0036667"/></geometry>
       <material name="handeye_black"><color rgba="0 0 0 1"/></material>
     </visual>
     <visual name="handeye_black_7">
-      <origin xyz="-0.00175 0.0964286 0.1125000" rpy="0 0 0"/>
-      <geometry><box size="0.0005 0.0171429 0.0085714"/></geometry>
+      <origin xyz="-0.00175 0.0508333 0.0618333" rpy="0 0 0"/>
+      <geometry><box size="0.0005 0.0036667 0.0036667"/></geometry>
       <material name="handeye_black"><color rgba="0 0 0 1"/></material>
     </visual>
     <visual name="handeye_black_8">
-      <origin xyz="-0.00175 0.0578571 0.1125000" rpy="0 0 0"/>
-      <geometry><box size="0.0005 0.0257143 0.0085714"/></geometry>
+      <origin xyz="-0.00175 0.0655000 0.0581667" rpy="0 0 0"/>
+      <geometry><box size="0.0005 0.0110000 0.0036667"/></geometry>
       <material name="handeye_black"><color rgba="0 0 0 1"/></material>
     </visual>
     <visual name="handeye_black_9">
-      <origin xyz="-0.00175 0.1007143 0.1039286" rpy="0 0 0"/>
-      <geometry><box size="0.0005 0.0085714 0.0085714"/></geometry>
+      <origin xyz="-0.00175 0.0508333 0.0581667" rpy="0 0 0"/>
+      <geometry><box size="0.0005 0.0036667 0.0036667"/></geometry>
       <material name="handeye_black"><color rgba="0 0 0 1"/></material>
     </visual>
     <visual name="handeye_black_10">
-      <origin xyz="-0.00175 0.0835714 0.1039286" rpy="0 0 0"/>
-      <geometry><box size="0.0005 0.0085714 0.0085714"/></geometry>
+      <origin xyz="-0.00175 0.0655000 0.0545000" rpy="0 0 0"/>
+      <geometry><box size="0.0005 0.0110000 0.0036667"/></geometry>
       <material name="handeye_black"><color rgba="0 0 0 1"/></material>
     </visual>
     <visual name="handeye_black_11">
-      <origin xyz="-0.00175 0.0664286 0.1039286" rpy="0 0 0"/>
-      <geometry><box size="0.0005 0.0085714 0.0085714"/></geometry>
+      <origin xyz="-0.00175 0.0526667 0.0545000" rpy="0 0 0"/>
+      <geometry><box size="0.0005 0.0073333 0.0036667"/></geometry>
       <material name="handeye_black"><color rgba="0 0 0 1"/></material>
     </visual>
     <visual name="handeye_black_12">
-      <origin xyz="-0.00175 0.0492857 0.1039286" rpy="0 0 0"/>
-      <geometry><box size="0.0005 0.0085714 0.0085714"/></geometry>
+      <origin xyz="-0.00175 0.0600000 0.0508333" rpy="0 0 0"/>
+      <geometry><box size="0.0005 0.0220000 0.0036667"/></geometry>
       <material name="handeye_black"><color rgba="0 0 0 1"/></material>
     </visual>
     <visual name="handeye_black_13">
-      <origin xyz="-0.00175 0.1007143 0.0953571" rpy="0 0 0"/>
-      <geometry><box size="0.0005 0.0085714 0.0085714"/></geometry>
+      <origin xyz="-0.00175 0.0300000 0.0600000" rpy="0 0 0"/>
+      <geometry><box size="0.0005 0.0300000 0.0300000"/></geometry>
       <material name="handeye_black"><color rgba="0 0 0 1"/></material>
     </visual>
     <visual name="handeye_black_14">
-      <origin xyz="-0.00175 0.0578571 0.0953571" rpy="0 0 0"/>
-      <geometry><box size="0.0005 0.0257143 0.0085714"/></geometry>
+      <origin xyz="-0.00175 0.0000000 0.0691667" rpy="0 0 0"/>
+      <geometry><box size="0.0005 0.0220000 0.0036667"/></geometry>
       <material name="handeye_black"><color rgba="0 0 0 1"/></material>
     </visual>
     <visual name="handeye_black_15">
-      <origin xyz="-0.00175 0.0750000 0.0867857" rpy="0 0 0"/>
-      <geometry><box size="0.0005 0.0600000 0.0085714"/></geometry>
+      <origin xyz="-0.00175 0.0000000 0.0655000" rpy="0 0 0"/>
+      <geometry><box size="0.0005 0.0220000 0.0036667"/></geometry>
       <material name="handeye_black"><color rgba="0 0 0 1"/></material>
     </visual>
     <visual name="handeye_black_16">
-      <origin xyz="-0.00175 0.0000000 0.1382143" rpy="0 0 0"/>
-      <geometry><box size="0.0005 0.0600000 0.0085714"/></geometry>
+      <origin xyz="-0.00175 0.0091667 0.0618333" rpy="0 0 0"/>
+      <geometry><box size="0.0005 0.0036667 0.0036667"/></geometry>
       <material name="handeye_black"><color rgba="0 0 0 1"/></material>
     </visual>
     <visual name="handeye_black_17">
-      <origin xyz="-0.00175 0.0085714 0.1296429" rpy="0 0 0"/>
-      <geometry><box size="0.0005 0.0428571 0.0085714"/></geometry>
+      <origin xyz="-0.00175 -0.0091667 0.0618333" rpy="0 0 0"/>
+      <geometry><box size="0.0005 0.0036667 0.0036667"/></geometry>
       <material name="handeye_black"><color rgba="0 0 0 1"/></material>
     </visual>
     <visual name="handeye_black_18">
-      <origin xyz="-0.00175 -0.0257143 0.1296429" rpy="0 0 0"/>
-      <geometry><box size="0.0005 0.0085714 0.0085714"/></geometry>
+      <origin xyz="-0.00175 0.0091667 0.0581667" rpy="0 0 0"/>
+      <geometry><box size="0.0005 0.0036667 0.0036667"/></geometry>
       <material name="handeye_black"><color rgba="0 0 0 1"/></material>
     </visual>
     <visual name="handeye_black_19">
-      <origin xyz="-0.00175 0.0257143 0.1210714" rpy="0 0 0"/>
-      <geometry><box size="0.0005 0.0085714 0.0085714"/></geometry>
+      <origin xyz="-0.00175 0.0000000 0.0581667" rpy="0 0 0"/>
+      <geometry><box size="0.0005 0.0073333 0.0036667"/></geometry>
       <material name="handeye_black"><color rgba="0 0 0 1"/></material>
     </visual>
     <visual name="handeye_black_20">
-      <origin xyz="-0.00175 -0.0128571 0.1210714" rpy="0 0 0"/>
-      <geometry><box size="0.0005 0.0342857 0.0085714"/></geometry>
+      <origin xyz="-0.00175 -0.0091667 0.0581667" rpy="0 0 0"/>
+      <geometry><box size="0.0005 0.0036667 0.0036667"/></geometry>
       <material name="handeye_black"><color rgba="0 0 0 1"/></material>
     </visual>
     <visual name="handeye_black_21">
-      <origin xyz="-0.00175 0.0085714 0.1125000" rpy="0 0 0"/>
-      <geometry><box size="0.0005 0.0428571 0.0085714"/></geometry>
+      <origin xyz="-0.00175 0.0091667 0.0545000" rpy="0 0 0"/>
+      <geometry><box size="0.0005 0.0036667 0.0036667"/></geometry>
       <material name="handeye_black"><color rgba="0 0 0 1"/></material>
     </visual>
     <visual name="handeye_black_22">
-      <origin xyz="-0.00175 -0.0257143 0.1125000" rpy="0 0 0"/>
-      <geometry><box size="0.0005 0.0085714 0.0085714"/></geometry>
+      <origin xyz="-0.00175 0.0018333 0.0545000" rpy="0 0 0"/>
+      <geometry><box size="0.0005 0.0036667 0.0036667"/></geometry>
       <material name="handeye_black"><color rgba="0 0 0 1"/></material>
     </visual>
     <visual name="handeye_black_23">
-      <origin xyz="-0.00175 0.0257143 0.1039286" rpy="0 0 0"/>
-      <geometry><box size="0.0005 0.0085714 0.0085714"/></geometry>
+      <origin xyz="-0.00175 -0.0073333 0.0545000" rpy="0 0 0"/>
+      <geometry><box size="0.0005 0.0073333 0.0036667"/></geometry>
       <material name="handeye_black"><color rgba="0 0 0 1"/></material>
     </visual>
     <visual name="handeye_black_24">
-      <origin xyz="-0.00175 0.0085714 0.1039286" rpy="0 0 0"/>
-      <geometry><box size="0.0005 0.0085714 0.0085714"/></geometry>
+      <origin xyz="-0.00175 0.0000000 0.0508333" rpy="0 0 0"/>
+      <geometry><box size="0.0005 0.0220000 0.0036667"/></geometry>
       <material name="handeye_black"><color rgba="0 0 0 1"/></material>
     </visual>
     <visual name="handeye_black_25">
-      <origin xyz="-0.00175 -0.0257143 0.1039286" rpy="0 0 0"/>
-      <geometry><box size="0.0005 0.0085714 0.0085714"/></geometry>
+      <origin xyz="-0.00175 -0.0300000 0.0600000" rpy="0 0 0"/>
+      <geometry><box size="0.0005 0.0300000 0.0300000"/></geometry>
       <material name="handeye_black"><color rgba="0 0 0 1"/></material>
     </visual>
     <visual name="handeye_black_26">
-      <origin xyz="-0.00175 0.0171429 0.0953571" rpy="0 0 0"/>
-      <geometry><box size="0.0005 0.0257143 0.0085714"/></geometry>
+      <origin xyz="-0.00175 -0.0600000 0.0691667" rpy="0 0 0"/>
+      <geometry><box size="0.0005 0.0220000 0.0036667"/></geometry>
       <material name="handeye_black"><color rgba="0 0 0 1"/></material>
     </visual>
     <visual name="handeye_black_27">
-      <origin xyz="-0.00175 -0.0214286 0.0953571" rpy="0 0 0"/>
-      <geometry><box size="0.0005 0.0171429 0.0085714"/></geometry>
+      <origin xyz="-0.00175 -0.0545000 0.0655000" rpy="0 0 0"/>
+      <geometry><box size="0.0005 0.0110000 0.0036667"/></geometry>
       <material name="handeye_black"><color rgba="0 0 0 1"/></material>
     </visual>
     <visual name="handeye_black_28">
-      <origin xyz="-0.00175 0.0000000 0.0867857" rpy="0 0 0"/>
-      <geometry><box size="0.0005 0.0600000 0.0085714"/></geometry>
+      <origin xyz="-0.00175 -0.0691667 0.0655000" rpy="0 0 0"/>
+      <geometry><box size="0.0005 0.0036667 0.0036667"/></geometry>
       <material name="handeye_black"><color rgba="0 0 0 1"/></material>
     </visual>
     <visual name="handeye_black_29">
-      <origin xyz="-0.00175 -0.0750000 0.1382143" rpy="0 0 0"/>
-      <geometry><box size="0.0005 0.0600000 0.0085714"/></geometry>
+      <origin xyz="-0.00175 -0.0545000 0.0618333" rpy="0 0 0"/>
+      <geometry><box size="0.0005 0.0110000 0.0036667"/></geometry>
       <material name="handeye_black"><color rgba="0 0 0 1"/></material>
     </visual>
     <visual name="handeye_black_30">
-      <origin xyz="-0.00175 -0.0492857 0.1296429" rpy="0 0 0"/>
-      <geometry><box size="0.0005 0.0085714 0.0085714"/></geometry>
+      <origin xyz="-0.00175 -0.0691667 0.0618333" rpy="0 0 0"/>
+      <geometry><box size="0.0005 0.0036667 0.0036667"/></geometry>
       <material name="handeye_black"><color rgba="0 0 0 1"/></material>
     </visual>
     <visual name="handeye_black_31">
-      <origin xyz="-0.00175 -0.0750000 0.1296429" rpy="0 0 0"/>
-      <geometry><box size="0.0005 0.0085714 0.0085714"/></geometry>
+      <origin xyz="-0.00175 -0.0545000 0.0581667" rpy="0 0 0"/>
+      <geometry><box size="0.0005 0.0110000 0.0036667"/></geometry>
       <material name="handeye_black"><color rgba="0 0 0 1"/></material>
     </visual>
     <visual name="handeye_black_32">
-      <origin xyz="-0.00175 -0.0964286 0.1296429" rpy="0 0 0"/>
-      <geometry><box size="0.0005 0.0171429 0.0085714"/></geometry>
+      <origin xyz="-0.00175 -0.0673333 0.0581667" rpy="0 0 0"/>
+      <geometry><box size="0.0005 0.0073333 0.0036667"/></geometry>
       <material name="handeye_black"><color rgba="0 0 0 1"/></material>
     </visual>
     <visual name="handeye_black_33">
-      <origin xyz="-0.00175 -0.0492857 0.1210714" rpy="0 0 0"/>
-      <geometry><box size="0.0005 0.0085714 0.0085714"/></geometry>
+      <origin xyz="-0.00175 -0.0508333 0.0545000" rpy="0 0 0"/>
+      <geometry><box size="0.0005 0.0036667 0.0036667"/></geometry>
       <material name="handeye_black"><color rgba="0 0 0 1"/></material>
     </visual>
     <visual name="handeye_black_34">
-      <origin xyz="-0.00175 -0.0964286 0.1210714" rpy="0 0 0"/>
-      <geometry><box size="0.0005 0.0171429 0.0085714"/></geometry>
+      <origin xyz="-0.00175 -0.0618333 0.0545000" rpy="0 0 0"/>
+      <geometry><box size="0.0005 0.0036667 0.0036667"/></geometry>
       <material name="handeye_black"><color rgba="0 0 0 1"/></material>
     </visual>
     <visual name="handeye_black_35">
-      <origin xyz="-0.00175 -0.0621429 0.1125000" rpy="0 0 0"/>
-      <geometry><box size="0.0005 0.0342857 0.0085714"/></geometry>
+      <origin xyz="-0.00175 -0.0691667 0.0545000" rpy="0 0 0"/>
+      <geometry><box size="0.0005 0.0036667 0.0036667"/></geometry>
       <material name="handeye_black"><color rgba="0 0 0 1"/></material>
     </visual>
     <visual name="handeye_black_36">
-      <origin xyz="-0.00175 -0.1007143 0.1125000" rpy="0 0 0"/>
-      <geometry><box size="0.0005 0.0085714 0.0085714"/></geometry>
+      <origin xyz="-0.00175 -0.0600000 0.0508333" rpy="0 0 0"/>
+      <geometry><box size="0.0005 0.0220000 0.0036667"/></geometry>
       <material name="handeye_black"><color rgba="0 0 0 1"/></material>
     </visual>
     <visual name="handeye_black_37">
-      <origin xyz="-0.00175 -0.0492857 0.1039286" rpy="0 0 0"/>
-      <geometry><box size="0.0005 0.0085714 0.0085714"/></geometry>
+      <origin xyz="-0.00175 -0.0900000 0.0600000" rpy="0 0 0"/>
+      <geometry><box size="0.0005 0.0300000 0.0300000"/></geometry>
       <material name="handeye_black"><color rgba="0 0 0 1"/></material>
     </visual>
     <visual name="handeye_black_38">
-      <origin xyz="-0.00175 -0.0664286 0.1039286" rpy="0 0 0"/>
-      <geometry><box size="0.0005 0.0085714 0.0085714"/></geometry>
+      <origin xyz="-0.00175 0.0900000 0.0391667" rpy="0 0 0"/>
+      <geometry><box size="0.0005 0.0220000 0.0036667"/></geometry>
       <material name="handeye_black"><color rgba="0 0 0 1"/></material>
     </visual>
     <visual name="handeye_black_39">
-      <origin xyz="-0.00175 -0.0964286 0.1039286" rpy="0 0 0"/>
-      <geometry><box size="0.0005 0.0171429 0.0085714"/></geometry>
+      <origin xyz="-0.00175 0.0991667 0.0355000" rpy="0 0 0"/>
+      <geometry><box size="0.0005 0.0036667 0.0036667"/></geometry>
       <material name="handeye_black"><color rgba="0 0 0 1"/></material>
     </visual>
     <visual name="handeye_black_40">
-      <origin xyz="-0.00175 -0.0492857 0.0953571" rpy="0 0 0"/>
-      <geometry><box size="0.0005 0.0085714 0.0085714"/></geometry>
+      <origin xyz="-0.00175 0.0900000 0.0355000" rpy="0 0 0"/>
+      <geometry><box size="0.0005 0.0073333 0.0036667"/></geometry>
       <material name="handeye_black"><color rgba="0 0 0 1"/></material>
     </visual>
     <visual name="handeye_black_41">
-      <origin xyz="-0.00175 -0.0835714 0.0953571" rpy="0 0 0"/>
-      <geometry><box size="0.0005 0.0085714 0.0085714"/></geometry>
+      <origin xyz="-0.00175 0.0808333 0.0355000" rpy="0 0 0"/>
+      <geometry><box size="0.0005 0.0036667 0.0036667"/></geometry>
       <material name="handeye_black"><color rgba="0 0 0 1"/></material>
     </visual>
     <visual name="handeye_black_42">
-      <origin xyz="-0.00175 -0.1007143 0.0953571" rpy="0 0 0"/>
-      <geometry><box size="0.0005 0.0085714 0.0085714"/></geometry>
+      <origin xyz="-0.00175 0.0991667 0.0318333" rpy="0 0 0"/>
+      <geometry><box size="0.0005 0.0036667 0.0036667"/></geometry>
       <material name="handeye_black"><color rgba="0 0 0 1"/></material>
     </visual>
     <visual name="handeye_black_43">
-      <origin xyz="-0.00175 -0.0750000 0.0867857" rpy="0 0 0"/>
-      <geometry><box size="0.0005 0.0600000 0.0085714"/></geometry>
+      <origin xyz="-0.00175 0.0900000 0.0318333" rpy="0 0 0"/>
+      <geometry><box size="0.0005 0.0073333 0.0036667"/></geometry>
       <material name="handeye_black"><color rgba="0 0 0 1"/></material>
     </visual>
     <visual name="handeye_black_44">
-      <origin xyz="-0.00175 0.0750000 0.0632143" rpy="0 0 0"/>
-      <geometry><box size="0.0005 0.0600000 0.0085714"/></geometry>
+      <origin xyz="-0.00175 0.0808333 0.0318333" rpy="0 0 0"/>
+      <geometry><box size="0.0005 0.0036667 0.0036667"/></geometry>
       <material name="handeye_black"><color rgba="0 0 0 1"/></material>
     </visual>
     <visual name="handeye_black_45">
-      <origin xyz="-0.00175 0.1007143 0.0546429" rpy="0 0 0"/>
-      <geometry><box size="0.0005 0.0085714 0.0085714"/></geometry>
+      <origin xyz="-0.00175 0.0973333 0.0281667" rpy="0 0 0"/>
+      <geometry><box size="0.0005 0.0073333 0.0036667"/></geometry>
       <material name="handeye_black"><color rgba="0 0 0 1"/></material>
     </visual>
     <visual name="handeye_black_46">
-      <origin xyz="-0.00175 0.0664286 0.0546429" rpy="0 0 0"/>
-      <geometry><box size="0.0005 0.0428571 0.0085714"/></geometry>
+      <origin xyz="-0.00175 0.0845000 0.0281667" rpy="0 0 0"/>
+      <geometry><box size="0.0005 0.0110000 0.0036667"/></geometry>
       <material name="handeye_black"><color rgba="0 0 0 1"/></material>
     </visual>
     <visual name="handeye_black_47">
-      <origin xyz="-0.00175 0.0921429 0.0460714" rpy="0 0 0"/>
-      <geometry><box size="0.0005 0.0257143 0.0085714"/></geometry>
+      <origin xyz="-0.00175 0.0973333 0.0245000" rpy="0 0 0"/>
+      <geometry><box size="0.0005 0.0073333 0.0036667"/></geometry>
       <material name="handeye_black"><color rgba="0 0 0 1"/></material>
     </visual>
     <visual name="handeye_black_48">
-      <origin xyz="-0.00175 0.0492857 0.0460714" rpy="0 0 0"/>
-      <geometry><box size="0.0005 0.0085714 0.0085714"/></geometry>
+      <origin xyz="-0.00175 0.0826667 0.0245000" rpy="0 0 0"/>
+      <geometry><box size="0.0005 0.0073333 0.0036667"/></geometry>
       <material name="handeye_black"><color rgba="0 0 0 1"/></material>
     </visual>
     <visual name="handeye_black_49">
-      <origin xyz="-0.00175 0.0921429 0.0375000" rpy="0 0 0"/>
-      <geometry><box size="0.0005 0.0257143 0.0085714"/></geometry>
+      <origin xyz="-0.00175 0.0900000 0.0208333" rpy="0 0 0"/>
+      <geometry><box size="0.0005 0.0220000 0.0036667"/></geometry>
       <material name="handeye_black"><color rgba="0 0 0 1"/></material>
     </visual>
     <visual name="handeye_black_50">
-      <origin xyz="-0.00175 0.0664286 0.0375000" rpy="0 0 0"/>
-      <geometry><box size="0.0005 0.0085714 0.0085714"/></geometry>
+      <origin xyz="-0.00175 0.0600000 0.0300000" rpy="0 0 0"/>
+      <geometry><box size="0.0005 0.0300000 0.0300000"/></geometry>
       <material name="handeye_black"><color rgba="0 0 0 1"/></material>
     </visual>
     <visual name="handeye_black_51">
-      <origin xyz="-0.00175 0.0492857 0.0375000" rpy="0 0 0"/>
-      <geometry><box size="0.0005 0.0085714 0.0085714"/></geometry>
+      <origin xyz="-0.00175 0.0300000 0.0391667" rpy="0 0 0"/>
+      <geometry><box size="0.0005 0.0220000 0.0036667"/></geometry>
       <material name="handeye_black"><color rgba="0 0 0 1"/></material>
     </visual>
     <visual name="handeye_black_52">
-      <origin xyz="-0.00175 0.0964286 0.0289286" rpy="0 0 0"/>
-      <geometry><box size="0.0005 0.0171429 0.0085714"/></geometry>
+      <origin xyz="-0.00175 0.0373333 0.0355000" rpy="0 0 0"/>
+      <geometry><box size="0.0005 0.0073333 0.0036667"/></geometry>
       <material name="handeye_black"><color rgba="0 0 0 1"/></material>
     </visual>
     <visual name="handeye_black_53">
-      <origin xyz="-0.00175 0.0492857 0.0289286" rpy="0 0 0"/>
-      <geometry><box size="0.0005 0.0085714 0.0085714"/></geometry>
+      <origin xyz="-0.00175 0.0281667 0.0355000" rpy="0 0 0"/>
+      <geometry><box size="0.0005 0.0036667 0.0036667"/></geometry>
       <material name="handeye_black"><color rgba="0 0 0 1"/></material>
     </visual>
     <visual name="handeye_black_54">
-      <origin xyz="-0.00175 0.1007143 0.0203571" rpy="0 0 0"/>
-      <geometry><box size="0.0005 0.0085714 0.0085714"/></geometry>
+      <origin xyz="-0.00175 0.0208333 0.0355000" rpy="0 0 0"/>
+      <geometry><box size="0.0005 0.0036667 0.0036667"/></geometry>
       <material name="handeye_black"><color rgba="0 0 0 1"/></material>
     </visual>
     <visual name="handeye_black_55">
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