Commit message: feat(handeye): 替换 ChArUco 标定板并完善仿真退出流程
将仿真标定板更新为 7×5、DICT_4X4_50、30 mm 方格和 22 mm Marker，完善自动检测与求解，并修复 Gazebo 和 MoveGroup 退出时的崩溃及强制终止提示。

File: src/zhishu_robot_description/urdf/head_camera_handeye.xacro (robot description, xacro)
@@ -35,6 +35,9 @@
             <horizontal_fov>1.0471975512</horizontal_fov>
             <image>
-              <width>640</width>
-              <height>480</height>
+              <!-- The real 22 mm markers are much smaller than the previous
+                   60 mm GridBoard markers.  Use enough pixels for reliable
+                   ChArUco corner interpolation in the headless renderer. -->
+              <width>1280</width>
+              <height>960</height>
               <format>R8G8B8</format>
             </image>
